File: extras/schematics/lora_tracker.kicad_pcb (KiCad board)
At the start: 2 copper layers, 40 x 95.2 mm, 18 parts, among them J1 Conn_Coaxial, J2 Conn_01x10_Female, J3 Conn_01x12_Female, J4 Conn_01x03_Female, U1 ESP32, U2 E22-400M30S, U3 Ai-Thinker-Ra-01

Commit message: Updates
Other:
- net class Default removed

Commit message: Updates
Parts:
- removed JP1, JP2, JP3: SolderJumper_3_Open, Jumper:SolderJumper-3_P1.3mm_Open_Pad1.0x1.5mm
- removed JP4, JP5, JP6, JP7, JP8: SolderJumper_2_Open, Jumper:SolderJumper-2_P1.3mm_Open_Pad1.0x1.5mm
- C1, C3: footprint Capacitor_SMD:C_0603_1608Metric_Pad1.05x0.95mm_HandSolder -> Capacitor_SMD:C_0603_1608Metric_Pad1.08x0.95mm_HandSolder
- J1: footprint Connector_Coaxial:SMA_Samtec_SMA-J-P-H-ST-EM1_EdgeMount -> Connector_Coaxial:SMA_Samtec_SMA-J-P-X-ST-EM1_EdgeMount
- U1: value ESP32 -> ESP32_30pin; footprint lora_tracker:esp32 devkit -> lora_tracker:esp32-devkit-wide_copy
- moved J4 5.48 mm to (78.7, 134.0), turned to 180 degrees
- moved U1 2.84 mm to (96.5, 88.3)
- moved J3 1.38 mm to (109.2, 125.1)
- moved J2 0.53 mm to (78.7, 117.3)
- turned J1 to 180 degrees
Connections:
- J2 pad 1: GPIO10 -> unconnected-(J2-Pad1)
- J2 pad 2: GPIO9 -> unconnected-(J2-Pad2)
- J3 pad 1: GPIO7 -> unconnected-(J3-Pad1)
- J3 pad 2: GPIO8 -> unconnected-(J3-Pad2)
- J3 pad 5: GPIO0 -> unconnected-(J3-Pad5)
- U1 pad 1: Net-(JP7-Pad2) -> EN
- U1 pad 10: GPIO26 -> NRST
- U1 pad 11: NRST -> BUSY
- U1 pad 12: BUSY -> DIO1
- U1 pad 13: DIO1 -> GPIO13
- U1 pad 14: Net-(JP4-Pad2) -> GND
- U1 pad 15: GPIO13 -> VCC
- U1 pad 16: GPIO9 -> 3v3
- U1 pad 17: GPIO10 -> GND
- U1 pad 18: Net-(JP5-Pad2) -> GPIO15
- U1 pad 19: VCC -> GPIO2
- U1 pad 2: EN -> GPIO36
- U1 pad 20: Net-(JP8-Pad1) -> GPIO4
- U1 pad 21: GPIO7 -> GPIO16
- U1 pad 22: GPIO8 -> GPIO17
- U1 pad 23: GPIO15 -> NSS
- U1 pad 24: GPIO2 -> SCK
- U1 pad 25: GPIO0 -> MISO
- U1 pad 26: GPIO4 -> GPIO21
- U1 pad 27: GPIO16 -> GPIO3
- U1 pad 28: GPIO17 -> GPIO1
- U1 pad 29: Net-(JP3-Pad1) -> GPIO22
- U1 pad 3: GPIO36 -> GPIO39
- U1 pad 30: Net-(JP2-Pad1) -> MOSI
- U1 pad 4: GPIO39 -> GPIO34
- U1 pad 5: GPIO34 -> GPIO35
- U1 pad 6: GPIO35 -> RXEN
- U1 pad 7: RXEN -> TXEN
- U1 pad 8: TXEN -> GPIO25
- U1 pad 9: GPIO25 -> GPIO26
- U2 pad 8: (no net) -> unconnected-(U2-Pad8)
- U3 pad 10: (no net) -> unconnected-(U3-Pad10)
- U3 pad 11: (no net) -> unconnected-(U3-Pad11)
- U3 pad 7: (no net) -> unconnected-(U3-Pad7)
- U3 pad 8: (no net) -> unconnected-(U3-Pad8)
Routing:
- net 3v3: track 124.1 -> 110.1 mm
- net GPIO9: track 13.5 -> 0.00 mm
- net GPIO13: track 13.3 -> 0.00 mm
- net GPIO10: track 12.9 -> 0.00 mm
- net VCC: track 86.9 -> 76.6 mm
- net GPIO7: track 9.57 -> 0.00 mm
- net GPIO8: track 8.87 -> 0.00 mm
- net GPIO22: track 8.86 -> 0.00 mm
- net GPIO0: track 8.58 -> 0.00 mm
- net GPIO15: track 8.58 -> 0.00 mm
- net Net-(JP1-Pad3): track 8.48 -> 0.00 mm
- net GPIO17: track 8.38 -> 0.00 mm
- net GPIO4: track 8.28 -> 0.00 mm
- net GPIO2: track 8.68 -> 0.54 mm
- net GPIO1: track 7.96 -> 0.00 mm
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
Commit message: Updated schematics
Parts:
- removed J2: Conn_01x10_Female, Connector_PinSocket_2.54mm:PinSocket_1x10_P2.54mm_Vertical
- removed J3: Conn_01x12_Female, Connector_PinSocket_2.54mm:PinSocket_1x12_P2.54mm_Vertical
- added C4: 100nF, Capacitor_SMD:C_0603_1608Metric_Pad1.08x0.95mm_HandSolder, F.Cu at (78.7, 90.5)
- added C5: 100nF, Capacitor_SMD:C_0603_1608Metric_Pad1.08x0.95mm_HandSolder, F.Cu at (95.2, 48.3)
- added C6: 100nF, Capacitor_SMD:C_0603_1608Metric_Pad1.08x0.95mm_HandSolder, B.Cu at (91.4, 133.3)
- added C7: 100nF, Capacitor_SMD:C_0603_1608Metric_Pad1.08x0.95mm_HandSolder, B.Cu at (105.5, 71.3)
- added C8: 0.1uF, Capacitor_SMD:C_0603_1608Metric_Pad1.08x0.95mm_HandSolder, B.Cu at (103.5, 83.8)
- added C9: 47uF, Capacitor_THT:CP_Radial_D4.0mm_P2.00mm, F.Cu at (84.5, 132.6)
- added R1: 100k, Resistor_SMD:R_0603_1608Metric_Pad0.98x0.95mm_HandSolder, B.Cu at (93.9, 133.3)
- added R2: 1k, Resistor_SMD:R_0603_1608Metric_Pad0.98x0.95mm_HandSolder, B.Cu at (103.6, 87.2)
- added R3: 10k, Resistor_SMD:R_0603_1608Metric_Pad0.98x0.95mm_HandSolder, F.Cu at (95.2, 45.7)
- added R4: 10k, Resistor_SMD:R_0603_1608Metric_Pad0.98x0.95mm_HandSolder, B.Cu at (105.4, 51.6)
- added R5: 10k, Resistor_SMD:R_0603_1608Metric_Pad0.98x0.95mm_HandSolder, B.Cu at (100.7, 51.7)
- added SW1: SW_Push, Button_Switch_THT:SW_Tactile_SKHH_Angled, F.Cu at (111.5, 83.5)
- added U4: INP441, lora_tracker:inp441, B.Cu at (82.5, 78.0)
- added U5: MAX98357A, lora_tracker:MAX98357A, B.Cu at (94.0, 109.3)
- added U6: SSD1306, lora_tracker:SSD1306, B.Cu at (93.3, 54.1)
- added U7: EC11, lora_tracker:ec11, F.Cu at (113.6, 46.3)
- J1: value Conn_Coaxial -> ANT
- J4: value Conn_01x03_Female -> Pwr
- U1: value ESP32_30pin -> ESP32; footprint lora_tracker:esp32-devkit-wide_copy -> lora_tracker:esp32-devkit-wide_30pin
- U3: value Ai-Thinker-Ra-01 -> RA-01
- moved C1 7.12 mm to (102.2, 83.8)
- moved C2 6.93 mm to (99.1, 87.0)
- moved C3 4.47 mm to (78.7, 61.4)
- moved U3 2.92 mm to (90.4, 65.4)
- moved U1 2.63 mm to (96.5, 90.9)
- moved U2 2.07 mm to (93.7, 64.8)
- moved J4 1.41 mm to (77.5, 134.6)
- moved J1 0.24 mm to (82.2, 45.9)
Connections:
- net Net-(J1-Pad1) renamed ANT
- net VCC renamed 5V
Routing:
- net GPIO16: track 0.69 -> 135.8 mm, vias 0 -> 2
- net 3v3: track 110.1 -> 218.5 mm, vias 0 -> 2
- net GPIO17: track 0.00 -> 86.9 mm
- net GPIO34: track 1.14 -> 75.4 mm
- net GPIO39: track 1.14 -> 71.7 mm, vias 0 -> 3
- net GPIO21: track 0.90 -> 60.4 mm, vias 0 -> 2
- net GPIO15: track 0.00 -> 49.9 mm, vias 0 -> 1
- net GPIO22: track 0.00 -> 49.6 mm, vias 0 -> 2
- net GPIO2: track 0.54 -> 49.0 mm, vias 0 -> 2
- net GPIO4: track 0.00 -> 42.7 mm, vias 0 -> 2
- net 5V: track 76.6 -> 116.6 mm, vias 0 -> 1
- net GPIO26: track 0.00 -> 33.2 mm, vias 0 -> 1
- net GPIO25: track 0.00 -> 25.9 mm, vias 0 -> 1
- net GPIO13: track 0.00 -> 22.7 mm
- net NRST: track 98.3 -> 86.2 mm, vias 2 -> 3
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
Commit message: Update schematics
Routing:
- net GPIO17: track 86.9 -> 86.2 mm
- net GND: track 0.65 -> 0.00 mm, vias 131 -> 132
- net GPIO26: vias 1 -> 0
Changed lines of the file:
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@@
     (property "Sheetname" "")
     (attr smd)
-    (fp_text reference "C5" (at 0 -1.43) (layer "F.SilkS")
+    (fp_text reference "C5" (at 0.146267 1.27) (layer "F.SilkS")
       (effects (font (size 1 1) (thickness 0.15)))
     )
@@
     (property "Sheetname" "")
     (attr smd)
-    (fp_text reference "R1" (at 0 1.43 90) (layer "B.SilkS")
+    (fp_text reference "R1" (at 0 -1.385 90) (layer "B.SilkS")
       (effects (font (size 1 1) (thickness 0.15)) (justify mirror))
     )
@@
     (property "Sheetname" "")
     (attr smd)
-    (fp_text reference "C7" (at 0 1.43) (layer "B.SilkS")
+    (fp_text reference "C7" (at -1.2 -2.4) (layer "B.SilkS")
       (effects (font (size 1 1) (thickness 0.15)) (justify mirror))
     )
@@
   (gr_line (start 113.665 43.18) (end 113.665 138.43) (layer "Edge.Cuts") (width 0.15))
   (gr_line (start 113.665 138.43) (end 73.66 138.43) (layer "Edge.Cuts") (width 0.15))
-  (segment (start 80.63 126.365) (end 81.28 126.365) (width 0.25) (layer "F.Cu") (net 1))
   (via (at 96.52 137.16) (size 0.8) (drill 0.4) (layers "F.Cu" "B.Cu") (net 1))
   (via (at 95.885 70.485) (size 0.8) (drill 0.4) (layers "F.Cu" "B.Cu") (free) (net 1))
@@
   (via (at 87.376 48.768) (size 0.8) (drill 0.4) (layers "F.Cu" "B.Cu") (net 1))
   (via (at 74.93 83.312) (size 0.8) (drill 0.4) (layers "F.Cu" "B.Cu") (net 1))
+  (via (at 78.74 124.46) (size 0.8) (drill 0.4) (layers "F.Cu" "B.Cu") (free) (net 1))
   (segment (start 97.628501 78.265103) (end 97.628501 76.77) (width 0.25) (layer "F.Cu") (net 2))
   (segment (start 90.895 84.998604) (end 97.628501 78.265103) (width 0.25) (layer "F.Cu") (net 2))
@@
   (segment (start 83.7325 108.6725) (end 91.44 100.965) (width 0.25) (layer "B.Cu") (net 3))
   (segment (start 89.26998 75.93498) (end 89.26998 74.02998) (width 0.25) (layer "F.Cu") (net 4))
-  (segment (start 102.708501 53.247499) (end 102.616 53.34) (width 0.25) (layer "F.Cu") (net 4))
   (segment (start 84.455 64.135) (end 82.694 64.135) (width 0.25) (layer "F.Cu") (net 4))
   (segment (start 89.26998 74.02998) (end 84.455 69.215) (width 0.25) (layer "F.Cu") (net 4))
@@
   (via (at 84.455 69.215) (size 0.8) (drill 0.4) (layers "F.Cu" "B.Cu") (net 4))
   (segment (start 84.455 69.215) (end 84.455 64.135) (width 0.25) (layer "B.Cu") (net 4))
-  (segment (start 84.455 60.505) (end 87.361396 57.598604) (width 0.25) (layer "B.Cu") (net 4))
-  (segment (start 89.085 57.598604) (end 91.438604 55.245) (width 0.25) (layer "B.Cu") (net 4))
+  (segment (start 92.073604 54.61) (end 101.981 54.61) (width 0.25) (layer "B.Cu") (net 4))
+  (segment (start 101.981 54.61) (end 102.616 55.245) (width 0.25) (layer "B.Cu") (net 4))
+  (segment (start 89.085 57.598604) (end 92.073604 54.61) (width 0.25) (layer "B.Cu") (net 4))
   (segment (start 87.361396 57.598604) (end 89.085 57.598604) (width 0.25) (layer "B.Cu") (net 4))
   (segment (start 84.455 64.135) (end 84.455 60.505) (width 0.25) (layer "B.Cu") (net 4))
-  (segment (start 91.438604 55.245) (end 102.616 55.245) (width 0.25) (layer "B.Cu") (net 4))
+  (segment (start 84.455 60.505) (end 87.361396 57.598604) (width 0.25) (layer "B.Cu") (net 4))
   (segment (start 81.28 118.8325) (end 89.71999 110.39251) (width 0.25) (layer "F.Cu") (net 5))
   (segment (start 85.725 66.675) (end 85.725 62.865) (width 0.25) (layer "F.Cu") (net 5))
@@
   (segment (start 105.248501 55.083501) (end 105.248501 52.77) (width 0.25) (layer "F.Cu") (net 5))
   (segment (start 85.725 62.865) (end 90.17 58.42) (width 0.25) (layer "F.Cu") (net 5))
-  (segment (start 82.694 66.675) (end 82.424 66.405) (width 0.25) (layer "F.Cu") (net 5))
   (segment (start 105.41 55.245) (end 105.248501 55.083501) (width 0.25) (layer "F.Cu") (net 5))
   (segment (start 89.71999 73.341643) (end 86.863347 70.485) (width 0.25) (layer "F.Cu") (net 5))
@@
   (segment (start 100.33 57.15) (end 97.628501 54.448501) (width 0.25) (layer "F.Cu") (net 10))
   (segment (start 99.52 62.405) (end 100.33 61.595) (width 0.25) (layer "F.Cu") (net 10))
-  (segment (start 97.536 52.832) (end 97.628501 52.739499) (width 0.25) (layer "F.Cu") (net 10))
   (segment (start 97.155 62.23) (end 98.249 62.23) (width 0.25) (layer "F.Cu") (net 10))
   (segment (start 98.249 62.23) (end 98.424 62.405) (width 0.25) (layer "F.Cu") (net 10))
@@
   (segment (start 95.885 123.9125) (end 81.28 123.9125) (width 0.25) (layer "B.Cu") (net 12))
   (segment (start 101.6 129.6275) (end 95.885 123.9125) (width 0.25) (layer "B.Cu") (net 12))
-  (via (at 81.28 113.7525) (size 0.8) (drill 0.4) (layers "F.Cu" "B.Cu") (net 13))
   (segment (start 102.87 129.894751) (end 102.87 129.360249) (width 0.25) (layer "B.Cu") (net 13))
   (segment (start 93.614751 120.105) (end 87.6325 120.105) (width 0.25) (layer "B.Cu") (net 13))
@@
   (segment (start 86.36 86.928423) (end 85.09 85.658423) (width 0.25) (layer "F.Cu") (net 20))
   (segment (start 86.36 107.95) (end 86.36 86.928423) (width 0.25) (layer "F.Cu") (net 20))
-  (segment (start 107.188 123.952) (end 107.061 123.825) (width 0.25) (layer "F.Cu") (net 20))
   (via (at 86.36 107.95) (size 0.8) (drill 0.4) (layers "F.Cu" "B.Cu") (net 20))
   (segment (start 106.68 123.9125) (end 102.3225 123.9125) (width 0.25) (layer "B.Cu") (net 20))
@@
   (segment (start 81.560249 130.81) (end 86.640249 125.73) (width 0.25) (layer "B.Cu") (net 22))
   (segment (start 76.745 62.456305) (end 76.745 125.994751) (width 0.25) (layer "B.Cu") (net 22))
-  (segment (start 106.68 113.284) (end 106.68 113.792) (width 0.25) (layer "F.Cu") (net 23))
-  (segment (start 106.68 113.792) (end 106.553 113.665) (width 0.25) (layer "F.Cu") (net 23))
   (segment (start 113.12 69.369695) (end 109.22 73.269695) (width 0.25) (layer "B.Cu") (net 23))
   (segment (start 110.49 113.03) (end 109.7675 113.7525) (width 0.25) (layer "B.Cu") (net 23))

Commit message: Update schematics
Parts:
- moved J1 0.35 mm to (82.5, 45.9)
Routing:
- net 3v3: track 218.5 -> 210.0 mm
- net GPIO26: track 33.2 -> 37.3 mm
- net GPIO16: track 135.8 -> 137.3 mm
- net GPIO34: track 75.4 -> 76.1 mm
- net GND: vias 132 -> 153

Commit message: Update schematics
Parts:
- added R6: 10k, Resistor_SMD:R_0603_1608Metric_Pad0.98x0.95mm_HandSolder, F.Cu at (78.1, 123.5)
- added R7: 10k, Resistor_SMD:R_0603_1608Metric_Pad0.98x0.95mm_HandSolder, F.Cu at (78.1, 119.4)
- J4: value Pwr -> Conn_01x03_Female; footprint Connector_PinSocket_2.54mm:PinSocket_1x03_P2.54mm_Vertical -> Connector_PinHeader_2.54mm:PinHeader_1x03_P2.54mm_Vertical
- moved J4 2.54 mm to (77.5, 132.1)
Connections:
- J4 pad 2: 3v3 -> 5V
- J4 pad 3: 5V -> Net-(R6-Pad1)
Routing:
- net GPIO36: track 0.00 -> 31.3 mm
- net Net-(R6-Pad1): track 0.00 -> 2.88 mm
- net 3v3: track 210.0 -> 212.6 mm
- net GPIO16: track 137.3 -> 136.7 mm
- net GND: track 0.00 -> 0.62 mm, vias 153 -> 157

Commit message: Update schematics
Parts:
- added C10: 100nF, Capacitor_SMD:C_0603_1608Metric_Pad1.08x0.95mm_HandSolder, F.Cu at (84.9, 95.8)
Routing:
- net GPIO36: track 31.3 -> 35.2 mm
- net GND: vias 157 -> 158
Changed lines of the file:
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@@
   (net 35 "GPIO2")
   (net 36 "Net-(R1-Pad1)")
-  (net 37 "Net-(R6-Pad1)")
+  (net 37 "Net-(J4-Pad3)")
   (footprint "Capacitor_SMD:CP_Elec_3x5.3" (layer "F.Cu")
     (at 99.06 86.995 -90)
@@
     )
   )
+  (footprint "Capacitor_SMD:C_0603_1608Metric_Pad1.08x0.95mm_HandSolder" (layer "F.Cu")
+    (at 84.855 95.8225 90)
+    (descr "Capacitor SMD 0603 (1608 Metric), square (rectangular) end terminal, IPC_7351 nominal with elongated pad for handsoldering. (Body size source: IPC-SM-782 page 76, https://www.pcb-3d.com/wordpress/wp-content/uploads/ipc-sm-782a_amendment_1_and_2.pdf), generated with kicad-footprint-generator")
+    (tags "capacitor handsolder")
+    (property "Sheetfile" "lora_tracker.kicad_sch")
+    (property "Sheetname" "")
+    (attr smd)
+    (fp_text reference "C10" (at 0 -1.43 90) (layer "F.SilkS")
+      (effects (font (size 1 1) (thickness 0.15)))
+    )
+    (fp_text value "100nF" (at 0 1.43 90) (layer "F.Fab")
+      (effects (font (size 1 1) (thickness 0.15)))
+    )
+    (fp_text user "${REFERENCE}" (at 0 0 90) (layer "F.Fab")
+      (effects (font (size 0.4 0.4) (thickness 0.06)))
+    )
+    (fp_line (start -0.146267 -0.51) (end 0.146267 -0.51) (layer "F.SilkS") (width 0.12))
+    (fp_line (start -0.146267 0.51) (end 0.146267 0.51) (layer "F.SilkS") (width 0.12))
+    (fp_line (start 1.65 0.73) (end -1.65 0.73) (layer "F.CrtYd") (width 0.05))
+    (fp_line (start -1.65 -0.73) (end 1.65 -0.73) (layer "F.CrtYd") (width 0.05))
+    (fp_line (start 1.65 -0.73) (end 1.65 0.73) (layer "F.CrtYd") (width 0.05))
+    (fp_line (start -1.65 0.73) (end -1.65 -0.73) (layer "F.CrtYd") (width 0.05))
+    (fp_line (start -0.8 0.4) (end -0.8 -0.4) (layer "F.Fab") (width 0.1))
+    (fp_line (start 0.8 -0.4) (end 0.8 0.4) (layer "F.Fab") (width 0.1))
+    (fp_line (start 0.8 0.4) (end -0.8 0.4) (layer "F.Fab") (width 0.1))
+    (fp_line (start -0.8 -0.4) (end 0.8 -0.4) (layer "F.Fab") (width 0.1))
+    (pad "1" smd roundrect (at -0.8625 0 90) (size 1.075 0.95) (layers "F.Cu" "F.Paste" "F.Mask") (roundrect_rratio 0.25)
+      (net 18 "GPIO36") (pintype "passive"))
+    (pad "2" smd roundrect (at 0.8625 0 90) (size 1.075 0.95) (layers "F.Cu" "F.Paste" "F.Mask") (roundrect_rratio 0.25)
+      (net 1 "GND") (pintype "passive"))
+    (model "${KICAD6_3DMODEL_DIR}/Capacitor_SMD.3dshapes/C_0603_1608Metric.wrl"
+      (offset (xyz 0 0 0))
+      (scale (xyz 1 1 1))
+      (rotate (xyz 0 0 0))
+    )
+  )
   (footprint "Resistor_SMD:R_0603_1608Metric_Pad0.98x0.95mm_HandSolder" (layer "F.Cu")
     (at 78.105 123.4675 90)
@@
     (fp_line (start 0.8 0.4125) (end -0.8 0.4125) (layer "F.Fab") (width 0.1))
     (pad "1" smd roundrect (at -0.9125 0 90) (size 0.975 0.95) (layers "F.Cu" "F.Paste" "F.Mask") (roundrect_rratio 0.25)
-      (net 37 "Net-(R6-Pad1)") (pintype "passive"))
+      (net 37 "Net-(J4-Pad3)") (pintype "passive"))
     (pad "2" smd roundrect (at 0.9125 0 90) (size 0.975 0.95) (layers "F.Cu" "F.Paste" "F.Mask") (roundrect_rratio 0.25)
       (net 18 "GPIO36") (pintype "passive"))
@@
       (net 33 "5V") (pinfunction "Pin_2") (pintype "passive"))
     (pad "3" thru_hole oval (at 0 5.08 180) (size 1.7 1.7) (drill 1) (layers *.Cu *.Mask)
-      (net 37 "Net-(R6-Pad1)") (pinfunction "Pin_3") (pintype "passive"))
+      (net 37 "Net-(J4-Pad3)") (pinfunction "Pin_3") (pintype "passive"))
     (model "${KICAD6_3DMODEL_DIR}/Connector_PinHeader_2.54mm.3dshapes/PinHeader_1x03_P2.54mm_Vertical.wrl"
       (offset (xyz 0 0 0))
@@
   (via (at 112.395 75.184) (size 0.8) (drill 0.4) (layers "F.Cu" "B.Cu") (net 1))
   (via (at 104.14 62.865) (size 0.8) (drill 0.4) (layers "F.Cu" "B.Cu") (free) (net 1))
-  (via (at 84.455 95.885) (size 0.8) (drill 0.4) (layers "F.Cu" "B.Cu") (free) (net 1))
   (via (at 93.98 70.485) (size 0.8) (drill 0.4) (layers "F.Cu" "B.Cu") (free) (net 1))
   (via (at 74.93 73.152) (size 0.8) (drill 0.4) (layers "F.Cu" "B.Cu") (net 1))
@@
   (via (at 99.06 134.62) (size 0.8) (drill 0.4) (layers "F.Cu" "B.Cu") (free) (net 1))
   (via (at 74.93 103.632) (size 0.8) (drill 0.4) (layers "F.Cu" "B.Cu") (net 1))
+  (via (at 83.185 93.98) (size 0.8) (drill 0.4) (layers "F.Cu" "B.Cu") (free) (net 1))
   (via (at 80.264 137.16) (size 0.8) (drill 0.4) (layers "F.Cu" "B.Cu") (net 1))
   (via (at 99.06 97.79) (size 0.8) (drill 0.4) (layers "F.Cu" "B.Cu") (free) (net 1))
@@
   (via (at 74.93 109.728) (size 0.8) (drill 0.4) (layers "F.Cu" "B.Cu") (net 1))
   (via (at 109.22 110.49) (size 0.8) (drill 0.4) (layers "F.Cu" "B.Cu") (free) (net 1))
+  (via (at 82.55 80.01) (size 0.8) (drill 0.4) (layers "F.Cu" "B.Cu") (free) (net 1))
   (via (at 112.395 80.01) (size 0.8) (drill 0.4) (layers "F.Cu" "B.Cu") (net 1))
   (via (at 87.884 46.736) (size 0.8) (drill 0.4) (layers "F.Cu" "B.Cu") (net 1))
@@
   (segment (start 78.015 113.575) (end 78.015 99.2375) (width 0.25) (layer "F.Cu") (net 18))
   (segment (start 78.105 122.555) (end 79.375 121.285) (width 0.25) (layer "F.Cu") (net 18))
+  (segment (start 83.35 96.685) (end 84.855 96.685) (width 0.25) (layer "F.Cu") (net 18))
   (segment (start 78.015 99.2375) (end 81.28 95.9725) (width 0.25) (layer "F.Cu") (net 18))
+  (segment (start 82.6375 95.9725) (end 83.35 96.685) (width 0.25) (layer "F.Cu") (net 18))
   (segment (start 78.105 122.555) (end 78.105 120.2925) (width 0.25) (layer "F.Cu") (net 18))
   (segment (start 79.375 121.285) (end 79.375 114.935) (width 0.25) (layer "F.Cu") (net 18))
+  (segment (start 81.28 95.9725) (end 82.6375 95.9725) (width 0.25) (layer "F.Cu") (net 18))
   (segment (start 86.36 86.928423) (end 85.09 85.658423) (width 0.25) (layer "F.Cu") (net 20))
   (segment (start 86.36 107.95) (end 86.36 86.928423) (width 0.25) (layer "F.Cu") (net 20))

Commit message: Update schematics
Parts:
- moved R6 4.14 mm to (78.7, 119.4)
- moved R7 3.86 mm to (78.7, 115.6)
- moved U7 3.15 mm to (110.5, 47.0)
- moved J4 2.62 mm to (78.1, 129.5)
- moved R3 1.95 mm to (93.3, 46.1)
- moved C5 1.91 mm to (93.3, 48.3)
Routing:
- net GPIO36: track 35.2 -> 29.1 mm
- net GPIO34: track 76.1 -> 72.0 mm
- net 3v3: track 212.6 -> 209.8 mm
- net GPIO17: track 86.2 -> 84.1 mm
- net GPIO16: track 136.7 -> 135.1 mm
- net Net-(J4-Pad3): track 2.88 -> 4.42 mm
- net GND: track 0.62 -> 0.58 mm, vias 158 -> 170
Other:
- outline, holes or cut-outs redrawn
