File: extras/schematics/lora_tracker.kicad_pcb (KiCad board)
At the start: 2 copper layers, 40 x 95.2 mm, 27 parts, among them J1 ANT, J4 Conn_01x03_Female, SW1 SW_Push, U1 ESP32, U2 E22-400M30S, U3 RA-01, U4 INP441, U5 MAX98357A, U6 SSD1306, U7 EC11

Commit message: Update schematics
Parts:
- moved SW1 0.64 mm to (110.8, 83.5)
Connections:
- SW1 pad : (no net) -> GND
Routing:
- net GPIO39: track 71.7 -> 71.0 mm
Changed lines of the file:
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@@
   )
   (footprint "Button_Switch_THT:SW_Tactile_SKHH_Angled" (layer "F.Cu")
-    (at 111.47 83.475 -90)
+    (at 110.835 83.475 -90)
     (descr "tactile switch 6mm ALPS SKHH right angle http://www.alps.com/prod/info/E/HTML/Tact/SnapIn/SKHH/SKHHLUA010.html")
     (tags "tactile switch 6mm ALPS SKHH right angle")
@@
     (fp_line (start 0.6 -2.55) (end 0.6 -5.85) (layer "F.Fab") (width 0.1))
     (fp_line (start 6 -2.55) (end -1.5 -2.55) (layer "F.Fab") (width 0.1))
-    (pad "" thru_hole circle (at 5.75 2.5 90) (size 2.2 2.2) (drill 1.3) (layers *.Cu *.Mask))
-    (pad "" thru_hole circle (at -1.25 2.5 90) (size 2.2 2.2) (drill 1.3) (layers *.Cu *.Mask))
+    (pad "" thru_hole circle (at 5.75 2.5 90) (size 2.2 2.2) (drill 1.3) (layers *.Cu *.Mask)
+      (net 1 "GND"))
+    (pad "" thru_hole circle (at -1.25 2.5 90) (size 2.2 2.2) (drill 1.3) (layers *.Cu *.Mask)
+      (net 1 "GND"))
     (pad "1" thru_hole circle (at 0 0 90) (size 1.7 1.7) (drill 1) (layers *.Cu *.Mask)
       (net 17 "GPIO39") (pinfunction "1") (pintype "passive"))
@@
   (via (at 85.09 109.22) (size 0.8) (drill 0.4) (layers "F.Cu" "B.Cu") (net 17))
   (via (at 91.44 115.57) (size 0.8) (drill 0.4) (layers "F.Cu" "B.Cu") (net 17))
+  (segment (start 109.22 85.09) (end 110.835 83.475) (width 0.25) (layer "B.Cu") (net 17))
   (segment (start 105.41 88.9) (end 105.41 88.04) (width 0.25) (layer "B.Cu") (net 17))
   (segment (start 104.411267 83.82) (end 105.681267 85.09) (width 0.25) (layer "B.Cu") (net 17))
   (segment (start 105.41 88.04) (end 104.555 87.185) (width 0.25) (layer "B.Cu") (net 17))
-  (segment (start 105.681267 85.09) (end 109.855 85.09) (width 0.25) (layer "B.Cu") (net 17))
   (segment (start 104.555 87.185) (end 104.555 85.945) (width 0.25) (layer "B.Cu") (net 17))
   (segment (start 85.09 109.22) (end 91.44 115.57) (width 0.25) (layer "B.Cu") (net 17))
   (segment (start 105.41 85.09) (end 105.681267 85.09) (width 0.25) (layer "B.Cu") (net 17))
-  (segment (start 109.855 85.09) (end 111.47 83.475) (width 0.25) (layer "B.Cu") (net 17))
   (segment (start 104.555 85.945) (end 105.41 85.09) (width 0.25) (layer "B.Cu") (net 17))
+  (segment (start 105.681267 85.09) (end 109.22 85.09) (width 0.25) (layer "B.Cu") (net 17))
   (segment (start 77.47 116.205) (end 77.47 113.485) (width 0.25) (layer "F.Cu") (net 18))
   (segment (start 77.7475 116.4825) (end 77.47 116.205) (width 0.25) (layer "F.Cu") (net 18))

Commit message: Update schematics
Parts:
- moved C4 6.11 mm to (78.1, 84.5), turned to 90 degrees
Routing:
- net 3v3: track 209.8 -> 206.6 mm
Changed lines of the file:
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@@
   )
   (footprint "Capacitor_SMD:C_0603_1608Metric_Pad1.08x0.95mm_HandSolder" (layer "F.Cu")
-    (at 78.74 90.53)
+    (at 78.105 84.455 90)
     (descr "Capacitor SMD 0603 (1608 Metric), square (rectangular) end terminal, IPC_7351 nominal with elongated pad for handsoldering. (Body size source: IPC-SM-782 page 76, https://www.pcb-3d.com/wordpress/wp-content/uploads/ipc-sm-782a_amendment_1_and_2.pdf), generated with kicad-footprint-generator")
     (tags "capacitor handsolder")
@@
     (property "Sheetname" "")
     (attr smd)
-    (fp_text reference "C4" (at 0 2.815) (layer "F.SilkS")
-      (effects (font (size 1 1) (thickness 0.15)))
-    )
-    (fp_text value "100nF" (at 0 1.43) (layer "F.Fab")
-      (effects (font (size 1 1) (thickness 0.15)))
-    )
-    (fp_text user "${REFERENCE}" (at 0 0) (layer "F.Fab")
+    (fp_text reference "C4" (at 0 2.815 90) (layer "F.SilkS")
+      (effects (font (size 1 1) (thickness 0.15)))
+    )
+    (fp_text value "100nF" (at 0 1.43 90) (layer "F.Fab")
+      (effects (font (size 1 1) (thickness 0.15)))
+    )
+    (fp_text user "${REFERENCE}" (at 0 0 90) (layer "F.Fab")
       (effects (font (size 0.4 0.4) (thickness 0.06)))
     )
@@
     (fp_line (start -0.8 0.4) (end -0.8 -0.4) (layer "F.Fab") (width 0.1))
     (fp_line (start 0.8 0.4) (end -0.8 0.4) (layer "F.Fab") (width 0.1))
-    (pad "1" smd roundrect (at -0.8625 0) (size 1.075 0.95) (layers "F.Cu" "F.Paste" "F.Mask") (roundrect_rratio 0.25)
+    (pad "1" smd roundrect (at -0.8625 0 90) (size 1.075 0.95) (layers "F.Cu" "F.Paste" "F.Mask") (roundrect_rratio 0.25)
       (net 11 "3v3") (pintype "passive"))
-    (pad "2" smd roundrect (at 0.8625 0) (size 1.075 0.95) (layers "F.Cu" "F.Paste" "F.Mask") (roundrect_rratio 0.25)
+    (pad "2" smd roundrect (at 0.8625 0 90) (size 1.075 0.95) (layers "F.Cu" "F.Paste" "F.Mask") (roundrect_rratio 0.25)
       (net 1 "GND") (pintype "passive"))
     (model "${KICAD6_3DMODEL_DIR}/Capacitor_SMD.3dshapes/C_0603_1608Metric.wrl"
@@
   (segment (start 91.44 85.09) (end 99.7825 93.4325) (width 0.25) (layer "B.Cu") (net 10))
   (segment (start 106.68 135.255) (end 106.045 135.89) (width 0.5) (layer "F.Cu") (net 11))
+  (segment (start 76.2 121.92) (end 76.2 90.17) (width 0.5) (layer "F.Cu") (net 11))
   (segment (start 88.685 56.797918) (end 88.685 51.015) (width 0.25) (layer "F.Cu") (net 11))
+  (segment (start 75.565 122.555) (end 76.2 121.92) (width 0.5) (layer "F.Cu") (net 11))
+  (segment (start 78.74 62.23) (end 77.47 62.23) (width 0.5) (layer "F.Cu") (net 11))
+  (segment (start 87.63 135.89) (end 87.21 136.31) (width 0.5) (layer "F.Cu") (net 11))
   (segment (start 106.68 128.9925) (end 109.7675 128.9925) (width 0.5) (layer "F.Cu") (net 11))
   (segment (start 93.98 50.8) (end 92.4825 49.3025) (width 0.25) (layer "F.Cu") (net 11))
   (segment (start 88.685 51.015) (end 91.44 48.26) (width 0.25) (layer "F.Cu") (net 11))
   (segment (start 109.7675 128.9925) (end 110.49 128.27) (width 0.5) (layer "F.Cu") (net 11))
-  (segment (start 75.565 132.08) (end 75.565 122.555) (width 0.5) (layer "F.Cu") (net 11))
-  (segment (start 75.565 122.555) (end 76.2 121.92) (width 0.5) (layer "F.Cu") (net 11))
   (segment (start 106.68 90.17) (end 104.14 90.17) (width 0.5) (layer "F.Cu") (net 11))
+  (segment (start 81.065 136.31) (end 77.47 132.715) (width 0.5) (layer "F.Cu") (net 11))
+  (segment (start 87.21 136.31) (end 81.065 136.31) (width 0.5) (layer "F.Cu") (net 11))
   (segment (start 91.44 48.26) (end 92.4825 48.26) (width 0.25) (layer "F.Cu") (net 11))
   (segment (start 76.2 90.17) (end 76.2 85.09) (width 0.5) (layer "F.Cu") (net 11))
@@
   (segment (start 80.01 85.658423) (end 76.768423 85.658423) (width 0.5) (layer "F.Cu") (net 11))
   (segment (start 78.74 62.23) (end 82.249 62.23) (width 0.5) (layer "F.Cu") (net 11))
-  (segment (start 87.21 136.31) (end 81.065 136.31) (width 0.5) (layer "F.Cu") (net 11))
   (segment (start 82.249 62.23) (end 82.424 62.405) (width 0.5) (layer "F.Cu") (net 11))
   (segment (start 92.4825 49.3025) (end 92.4825 48.26) (width 0.25) (layer "F.Cu") (net 11))
-  (segment (start 81.065 136.31) (end 78.74 133.985) (width 0.5) (layer "F.Cu") (net 11))
+  (segment (start 75.565 132.08) (end 75.565 122.555) (width 0.5) (layer "F.Cu") (net 11))
+  (segment (start 77.47 62.23) (end 76.2 63.5) (width 0.5) (layer "F.Cu") (net 11))
   (segment (start 106.045 135.89) (end 87.63 135.89) (width 0.5) (layer "F.Cu") (net 11))
-  (segment (start 78.74 132.08) (end 75.565 132.08) (width 0.5) (layer "F.Cu") (net 11))
-  (segment (start 87.63 135.89) (end 87.21 136.31) (width 0.5) (layer "F.Cu") (net 11))
-  (segment (start 76.56 90.53) (end 76.2 90.17) (width 0.25) (layer "F.Cu") (net 11))
   (segment (start 76.768423 85.658423) (end 76.2 85.09) (width 0.5) (layer "F.Cu") (net 11))
-  (segment (start 77.8775 90.53) (end 76.56 90.53) (width 0.5) (layer "F.Cu") (net 11))
-  (segment (start 76.2 121.92) (end 76.2 90.17) (width 0.5) (layer "F.Cu") (net 11))
-  (segment (start 76.2 62.4575) (end 78.5125 62.4575) (width 0.5) (layer "F.Cu") (net 11))
+  (segment (start 77.47 132.715) (end 76.2 132.715) (width 0.5) (layer "F.Cu") (net 11))
+  (segment (start 76.2 85.09) (end 76.2 63.5) (width 0.5) (layer "F.Cu") (net 11))
   (segment (start 83.077918 62.405) (end 88.685 56.797918) (width 0.25) (layer "F.Cu") (net 11))
-  (segment (start 106.68 128.9925) (end 106.68 135.255) (width 0.5) (layer "F.Cu") (net 11))
   (segment (start 92.4825 46.1825) (end 92.4325 46.1325) (width 0.25) (layer "F.Cu") (net 11))
   (segment (start 78.5125 62.4575) (end 78.74 62.23) (width 0.5) (layer "F.Cu") (net 11))
-  (segment (start 76.2 85.09) (end 76.2 62.4575) (width 0.5) (layer "F.Cu") (net 11))
   (segment (start 110.49 93.98) (end 106.68 90.17) (width 0.5) (layer "F.Cu") (net 11))
-  (segment (start 78.74 133.985) (end 78.74 132.08) (width 0.5) (layer "F.Cu") (net 11))
   (segment (start 82.424 62.405) (end 83.077918 62.405) (width 0.5) (layer "F.Cu") (net 11))
   (segment (start 110.49 128.27) (end 110.49 93.98) (width 0.5) (layer "F.Cu") (net 11))
+  (segment (start 76.2 132.715) (end 75.565 132.08) (width 0.5) (layer "F.Cu") (net 11))
+  (segment (start 106.68 128.9925) (end 106.68 135.255) (width 0.5) (layer "F.Cu") (net 11))
   (via (at 104.14 90.17) (size 0.8) (drill 0.4) (layers "F.Cu" "B.Cu") (net 11))
   (via (at 93.98 50.8) (size 0.8) (drill 0.4) (layers "F.Cu" "B.Cu") (net 11))

Commit message: Update schematics
Connections:
- SW1 pad : GND -> (no net)
- U1 pad 1: EN -> unconnected-(U1-Pad1)
- U1 pad 27: GPIO3 -> unconnected-(U1-Pad27)
- U1 pad 28: GPIO1 -> unconnected-(U1-Pad28)
- U1 pad 5: GPIO35 -> unconnected-(U1-Pad5)
Changed lines of the file:
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@@
   (net 13 "GPIO26")
   (net 14 "GPIO25")
-  (net 15 "GPIO35")
+  (net 15 "unconnected-(U1-Pad1)")
   (net 16 "GPIO34")
   (net 17 "GPIO39")
   (net 18 "GPIO36")
-  (net 19 "EN")
+  (net 19 "unconnected-(U1-Pad5)")
   (net 20 "GPIO15")
   (net 21 "GPIO4")
@@
   (net 23 "GPIO17")
   (net 24 "GPIO21")
-  (net 25 "GPIO3")
-  (net 26 "GPIO1")
+  (net 25 "unconnected-(U1-Pad27)")
+  (net 26 "unconnected-(U1-Pad28)")
   (net 27 "GPIO22")
   (net 28 "unconnected-(U2-Pad8)")
@@
     (fp_line (start 0.6 -2.55) (end 0.6 -5.85) (layer "F.Fab") (width 0.1))
     (fp_line (start 6 -2.55) (end -1.5 -2.55) (layer "F.Fab") (width 0.1))
-    (pad "" thru_hole circle (at 5.75 2.5 90) (size 2.2 2.2) (drill 1.3) (layers *.Cu *.Mask)
-      (net 1 "GND"))
-    (pad "" thru_hole circle (at -1.25 2.5 90) (size 2.2 2.2) (drill 1.3) (layers *.Cu *.Mask)
-      (net 1 "GND"))
+    (pad "" thru_hole circle (at 5.75 2.5 90) (size 2.2 2.2) (drill 1.3) (layers *.Cu *.Mask))
+    (pad "" thru_hole circle (at -1.25 2.5 90) (size 2.2 2.2) (drill 1.3) (layers *.Cu *.Mask))
     (pad "1" thru_hole circle (at 0 0 90) (size 1.7 1.7) (drill 1) (layers *.Cu *.Mask)
       (net 17 "GPIO39") (pinfunction "1") (pintype "passive"))
@@
     (property "Sheetname" "")
     (attr smd)
-    (fp_text reference "C4" (at 0 2.815 90) (layer "F.SilkS")
+    (fp_text reference "C4" (at -3.175 0 90) (layer "F.SilkS")
       (effects (font (size 1 1) (thickness 0.15)))
     )
@@
     (fp_line (start -13.97 40.64) (end 8.89 40.64) (layer "F.SilkS") (width 0.15))
     (pad "1" thru_hole circle (at -15.24 2.54) (size 1.524 1.524) (drill 0.762) (layers *.Cu *.Mask)
-      (net 19 "EN") (pinfunction "EN") (pintype "input"))
+      (net 15 "unconnected-(U1-Pad1)") (pinfunction "EN") (pintype "input+no_connect"))
     (pad "2" thru_hole circle (at -15.24 5.08) (size 1.524 1.524) (drill 0.762) (layers *.Cu *.Mask)
       (net 18 "GPIO36") (pinfunction "VP/36") (pintype "input"))
@@
       (net 16 "GPIO34") (pinfunction "GPIO34") (pintype "input"))
     (pad "5" thru_hole circle (at -15.24 12.7) (size 1.524 1.524) (drill 0.762) (layers *.Cu *.Mask)
-      (net 15 "GPIO35") (pinfunction "GPIO35") (pintype "input"))
+      (net 19 "unconnected-(U1-Pad5)") (pinfunction "GPIO35") (pintype "input+no_connect"))
     (pad "6" thru_hole circle (at -15.24 15.24) (size 1.524 1.524) (drill 0.762) (layers *.Cu *.Mask)
       (net 2 "RXEN") (pinfunction "GPIO32") (pintype "input"))
@@
       (net 24 "GPIO21") (pinfunction "GPIO21") (pintype "input"))
     (pad "27" thru_hole circle (at 10.16 10.16) (size 1.524 1.524) (drill 0.762) (layers *.Cu *.Mask)
-      (net 25 "GPIO3") (pinfunction "RX0/03") (pintype "input"))
+      (net 25 "unconnected-(U1-Pad27)") (pinfunction "RX0/03") (pintype "input+no_connect"))
     (pad "28" thru_hole circle (at 10.16 7.62) (size 1.524 1.524) (drill 0.762) (layers *.Cu *.Mask)
-      (net 26 "GPIO1") (pinfunction "TX0/01") (pintype "input"))
+      (net 26 "unconnected-(U1-Pad28)") (pinfunction "TX0/01") (pintype "input+no_connect"))
     (pad "29" thru_hole circle (at 10.16 5.08) (size 1.524 1.524) (drill 0.762) (layers *.Cu *.Mask)
       (net 27 "GPIO22") (pinfunction "GPIO22") (pintype "input"))
@@
   (segment (start 106.68 135.255) (end 106.045 135.89) (width 0.5) (layer "F.Cu") (net 11))
   (segment (start 76.2 121.92) (end 76.2 90.17) (width 0.5) (layer "F.Cu") (net 11))
+  (segment (start 83.077918 62.405) (end 88.685 56.797918) (width 0.25) (layer "F.Cu") (net 11))
   (segment (start 88.685 56.797918) (end 88.685 51.015) (width 0.25) (layer "F.Cu") (net 11))
   (segment (start 75.565 122.555) (end 76.2 121.92) (width 0.5) (layer "F.Cu") (net 11))
@@
   (segment (start 92.4825 48.26) (end 92.4825 46.1825) (width 0.25) (layer "F.Cu") (net 11))
   (segment (start 80.01 85.658423) (end 76.768423 85.658423) (width 0.5) (layer "F.Cu") (net 11))
-  (segment (start 78.74 62.23) (end 82.249 62.23) (width 0.5) (layer "F.Cu") (net 11))
-  (segment (start 82.249 62.23) (end 82.424 62.405) (width 0.5) (layer "F.Cu") (net 11))
   (segment (start 92.4825 49.3025) (end 92.4825 48.26) (width 0.25) (layer "F.Cu") (net 11))
   (segment (start 75.565 132.08) (end 75.565 122.555) (width 0.5) (layer "F.Cu") (net 11))
   (segment (start 77.47 62.23) (end 76.2 63.5) (width 0.5) (layer "F.Cu") (net 11))
+  (segment (start 82.424 62.405) (end 83.077918 62.405) (width 0.5) (layer "F.Cu") (net 11))
   (segment (start 106.045 135.89) (end 87.63 135.89) (width 0.5) (layer "F.Cu") (net 11))
   (segment (start 76.768423 85.658423) (end 76.2 85.09) (width 0.5) (layer "F.Cu") (net 11))
   (segment (start 77.47 132.715) (end 76.2 132.715) (width 0.5) (layer "F.Cu") (net 11))
   (segment (start 76.2 85.09) (end 76.2 63.5) (width 0.5) (layer "F.Cu") (net 11))
-  (segment (start 83.077918 62.405) (end 88.685 56.797918) (width 0.25) (layer "F.Cu") (net 11))
+  (segment (start 82.249 62.23) (end 82.424 62.405) (width 0.5) (layer "F.Cu") (net 11))
   (segment (start 92.4825 46.1825) (end 92.4325 46.1325) (width 0.25) (layer "F.Cu") (net 11))
-  (segment (start 78.5125 62.4575) (end 78.74 62.23) (width 0.5) (layer "F.Cu") (net 11))
+  (segment (start 78.74 62.23) (end 82.249 62.23) (width 0.5) (layer "F.Cu") (net 11))
   (segment (start 110.49 93.98) (end 106.68 90.17) (width 0.5) (layer "F.Cu") (net 11))
-  (segment (start 82.424 62.405) (end 83.077918 62.405) (width 0.5) (layer "F.Cu") (net 11))
   (segment (start 110.49 128.27) (end 110.49 93.98) (width 0.5) (layer "F.Cu") (net 11))
   (segment (start 76.2 132.715) (end 75.565 132.08) (width 0.5) (layer "F.Cu") (net 11))
@@
   (segment (start 90.805 45.72) (end 91.44 45.085) (width 0.25) (layer "F.Cu") (net 22))
   (segment (start 90.805 47.625) (end 90.805 45.72) (width 0.25) (layer "F.Cu") (net 22))
-  (segment (start 94.3875 45.77) (end 94.3375 45.72) (width 0.5) (layer "F.Cu") (net 22))
   (segment (start 96.52 125.73) (end 97.2425 125.73) (width 0.25) (layer "F.Cu") (net 22))
   (segment (start 97.2425 125.73) (end 106.68 116.2925) (width 0.25) (layer "F.Cu") (net 22))
@@
   (via (at 89.535 48.895) (size 0.8) (drill 0.4) (layers "F.Cu" "B.Cu") (net 22))
   (via (at 96.52 125.73) (size 0.8) (drill 0.4) (layers "F.Cu" "B.Cu") (net 22))
+  (segment (start 76.835 61.595) (end 89.535 48.895) (width 0.25) (layer "B.Cu") (net 22))
+  (segment (start 76.835 120.65) (end 76.835 61.595) (width 0.25) (layer "B.Cu") (net 22))
+  (segment (start 80.01 130.81) (end 79.375 130.175) (width 0.25) (layer "B.Cu") (net 22))
+  (segment (start 81.560249 130.81) (end 80.01 130.81) (width 0.25) (layer "B.Cu") (net 22))
+  (segment (start 79.375 130.175) (end 79.375 123.19) (width 0.25) (layer "B.Cu") (net 22))
+  (segment (start 79.375 123.19) (end 76.835 120.65) (width 0.25) (layer "B.Cu") (net 22))
   (segment (start 96.52 125.73) (end 86.640249 125.73) (width 0.25) (layer "B.Cu") (net 22))
-  (segment (start 76.835 61.595) (end 89.535 48.895) (width 0.25) (layer "B.Cu") (net 22))
-  (segment (start 80.01 130.81) (end 79.375 130.175) (width 0.25) (layer "B.Cu") (net 22))
   (segment (start 86.640249 125.73) (end 81.560249 130.81) (width 0.25) (layer "B.Cu") (net 22))
-  (segment (start 76.835 123.19) (end 76.835 61.595) (width 0.25) (layer "B.Cu") (net 22))
-  (segment (start 79.375 125.73) (end 76.835 123.19) (width 0.25) (layer "B.Cu") (net 22))
-  (segment (start 79.375 130.175) (end 79.375 125.73) (width 0.25) (layer "B.Cu") (net 22))
-  (segment (start 81.560249 130.81) (end 80.01 130.81) (width 0.25) (layer "B.Cu") (net 22))
   (segment (start 104.7675 45.085) (end 104.14 45.7125) (width 0.25) (layer "B.Cu") (net 23))
   (segment (start 113.12 69.369695) (end 109.22 73.269695) (width 0.25) (layer "B.Cu") (net 23))
@@
   (segment (start 82.424 58.405) (end 82.424 52.785499) (width 1) (layer "F.Cu") (net 34))
   (segment (start 82.424 52.785499) (end 82.408501 52.77) (width 0.25) (layer "F.Cu") (net 34))
-  (segment (start 82.408501 45.946001) (end 82.2 45.7375) (width 0.25) (layer "F.Cu") (net 34))
   (segment (start 87.63 106.68) (end 87.63 92.71) (width 0.25) (layer "F.Cu") (net 35))
   (via (at 87.63 92.71) (size 0.8) (drill 0.4) (layers "F.Cu" "B.Cu") (net 35))

Commit message: Update schematics
Parts:
- moved C2 2.54 mm to (99.1, 84.5)
- moved U4 2.54 mm to (85.1, 78.0)
- moved SW1 1.91 mm to (110.8, 81.6)
- moved C1 1.53 mm to (103.5, 83.0)
- moved C9 0.47 mm to (84.5, 133.1)
- renumbered U7 to SW2
Connections:
- SW1 pad : (no net) -> GND
Routing:
- net 5V: track 116.7 -> 113.3 mm
- net GPIO4: track 42.7 -> 41.3 mm
- net GPIO39: track 71.0 -> 71.8 mm
- net 3v3: track 206.3 -> 207.0 mm
- net GND: vias 170 -> 175

Commit message: Update schematics
Parts:
- R3: moved to B.Cu
- moved R3 2.68 mm to (90.8, 47.0), turned to -90 degrees
- moved C5 2.54 mm to (90.8, 48.3), turned to 90 degrees
- moved SW2 0.96 mm to (109.8, 46.3)
Routing:
- net GPIO17: track 84.1 -> 80.4 mm
- net 3v3: track 207.0 -> 209.5 mm, vias 2 -> 3
- net GPIO16: track 135.0 -> 133.6 mm, vias 2 -> 1
- net GND: track 0.58 -> 0.05 mm, vias 175 -> 174

Commit message: Update schematics
Parts:
- U5: moved to F.Cu
- moved C6 5.08 mm to (96.5, 133.3)
- moved R3 1.27 mm to (90.8, 48.3)
- turned U5 to 0 degrees
Routing:
- net GPIO26: track 37.3 -> 20.1 mm, vias 0 -> 1
- net 5V: track 113.3 -> 125.4 mm
- net GPIO13: track 22.7 -> 14.5 mm, vias 0 -> 1
- net GPIO25: track 25.9 -> 23.8 mm
- net 3v3: track 209.5 -> 207.7 mm
- net GPIO16: track 133.6 -> 132.4 mm
- net GND: vias 174 -> 170

Commit message: Update schematics
Parts:
- added ?: , , F.Cu at (99.7, 109.9)
- added ?: , , F.Cu at (97.2, 109.9)
- added C11: 100nF, Capacitor_SMD:C_0603_1608Metric_Pad1.08x0.95mm_HandSolder, F.Cu at (99.1, 99.7)
- added U7: ATGM336H, lora_tracker:ATGM336H, F.Cu at (97.8, 89.5)
- moved C7 0.70 mm to (104.8, 71.3)
Connections:
- SW1 pad : GND -> (no net)
- U1 pad 27: unconnected-(U1-Pad27) -> GPIO3
- U1 pad 28: unconnected-(U1-Pad28) -> GPIO1
Routing:
- net 3v3: track 207.7 -> 224.9 mm
- net GPIO3: track 0.00 -> 4.37 mm
- net GPIO1: track 0.00 -> 4.37 mm
- net GPIO17: track 80.4 -> 82.5 mm, vias 0 -> 2
- net GPIO21: track 60.4 -> 61.9 mm
- net GPIO22: track 49.6 -> 50.8 mm
- net GND: vias 170 -> 168
Other:
- board text added: "+"
- board text added: "-"
- board text added: "SPK"
- board text added: "_"

Commit message: Update schematics
Routing:
- net GND: vias 168 -> 169
Other:
- board text added: "+5V"
- board text added: "BS"
- board text added: "GND"
Changed lines of the file:
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@@
     (effects (font (size 1.5 1.5) (thickness 0.3)) (justify mirror))
+  )
+  (gr_text "+5V" (at 75.565 127 90) (layer "F.SilkS")
+    (effects (font (size 1 1) (thickness 0.25)))
+  )
+  (gr_text "BS" (at 75.565 123.19 90) (layer "F.SilkS")
+    (effects (font (size 1 1) (thickness 0.25)))
   )
   (gr_text "SPK" (at 98.425 107.315) (layer "F.SilkS")
@@
   (gr_text "-" (at 95.885 107.95) (layer "F.SilkS")
     (effects (font (size 1 1) (thickness 0.15)))
+  )
+  (gr_text "GND" (at 75.565 130.81 90) (layer "F.SilkS")
+    (effects (font (size 1 1) (thickness 0.25)))
   )
   (segment (start 94.2575 46.1325) (end 94.2575 46.0775) (width 0.25) (layer "F.Cu") (net 1))
@@
   (via (at 74.93 95.504) (size 0.8) (drill 0.4) (layers "F.Cu" "B.Cu") (net 1))
   (via (at 74.93 93.472) (size 0.8) (drill 0.4) (layers "F.Cu" "B.Cu") (net 1))
+  (via (at 99.06 127) (size 0.8) (drill 0.4) (layers "F.Cu" "B.Cu") (free) (net 1))
   (via (at 112.395 117.856) (size 0.8) (drill 0.4) (layers "F.Cu" "B.Cu") (net 1))
   (via (at 97.79 122.555) (size 0.8) (drill 0.4) (layers "F.Cu" "B.Cu") (free) (net 1))
