File: extras/schematics/lora_tracker.kicad_pcb (KiCad board)
At the start: 2 copper layers, 40 x 95.2 mm, 34 parts, among them J1 ANT, J2 Conn_01x02, J4 Conn_01x03_Female, SW1 SW_Push, SW2 EC11, U1 ESP32, U2 E22-400M30S, U3 RA-01, U4 INP441, U5 MAX98357A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

Commit message: Update schematics
Routing:
- net GPIO17: track 82.5 -> 93.2 mm
- net GPIO21: track 61.9 -> 65.2 mm
- net MISO: track 72.4 -> 74.0 mm
- net GPIO22: track 50.8 -> 51.6 mm
- net GND: vias 146 -> 152

Commit message: Update schematics
Parts:
- removed ? (x2): , 
- removed REF** (x2): SolderWirePad_1x01_SMD_1x2mm, Connector_Wire:SolderWirePad_1x01_SMD_1x2mm
Connections:
- SW1 pad : (no net) -> GND
Changed lines of the file:
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@@
   (net 37 "Net-(J4-Pad3)")
   (net 38 "unconnected-(U7-Pad1)")
-  (net 39 "Net-(U5-Pad9)")
-  (net 40 "Net-(U5-Pad8)")
+  (net 39 "Net-(J2-Pad1)")
+  (net 40 "Net-(J2-Pad2)")
   (footprint "Capacitor_SMD:CP_Elec_3x5.3" (layer "F.Cu")
     (at 99.06 84.455 -90)
@@
     (fp_line (start 0.6 -2.55) (end 0.6 -5.85) (layer "F.Fab") (width 0.1))
     (fp_line (start 6 -2.55) (end -1.5 -2.55) (layer "F.Fab") (width 0.1))
-    (pad "" thru_hole circle (at 5.75 2.5 90) (size 2.2 2.2) (drill 1.3) (layers *.Cu *.Mask))
-    (pad "" thru_hole circle (at -1.25 2.5 90) (size 2.2 2.2) (drill 1.3) (layers *.Cu *.Mask))
+    (pad "" thru_hole circle (at 5.75 2.5 90) (size 2.2 2.2) (drill 1.3) (layers *.Cu *.Mask)
+      (net 1 "GND"))
+    (pad "" thru_hole circle (at -1.25 2.5 90) (size 2.2 2.2) (drill 1.3) (layers *.Cu *.Mask)
+      (net 1 "GND"))
     (pad "1" thru_hole circle (at 0 0 90) (size 1.7 1.7) (drill 1) (layers *.Cu *.Mask)
       (net 17 "GPIO39") (pinfunction "1") (pintype "passive"))
@@
       (net 33 "5V") (pinfunction "VIN") (pintype "power_in"))
     (pad "8" thru_hole circle (at 1.905 6.985) (size 1.524 1.524) (drill 0.762) (layers *.Cu *.Mask)
-      (net 40 "Net-(U5-Pad8)") (pinfunction "SPK+") (pintype "output"))
+      (net 40 "Net-(J2-Pad2)") (pinfunction "SPK+") (pintype "output"))
     (pad "9" thru_hole circle (at -1.905 6.985) (size 1.524 1.524) (drill 0.762) (layers *.Cu *.Mask)
-      (net 39 "Net-(U5-Pad9)") (pinfunction "SPK-") (pintype "output"))
+      (net 39 "Net-(J2-Pad1)") (pinfunction "SPK-") (pintype "output"))
   )
   (footprint "Capacitor_SMD:C_0603_1608Metric_Pad1.08x0.95mm_HandSolder" (layer "F.Cu")
@@
       (net 10 "MOSI") (pinfunction "GPIO23") (pintype "bidirectional"))
   )
-  (footprint "Connector_Wire:SolderWirePad_1x01_SMD_1x2mm" (layer "F.Cu")
-    (at 112.395 71.12)
-    (descr "Wire Pad, Square, SMD Pad,  1mm x 2mm,")
-    (tags "MesurementPoint Square SMDPad 1mmx2mm ")
-    (attr exclude_from_pos_files exclude_from_bom)
-    (fp_text reference "REF**" (at 0 -2.54) (layer "F.SilkS") hide
-      (effects (font (size 1 1) (thickness 0.15)))
-    )
-    (fp_text value "SolderWirePad_1x01_SMD_1x2mm" (at 0 2.54) (layer "F.Fab") hide
-      (effects (font (size 1 1) (thickness 0.15)))
-    )
-    (fp_text user "${REFERENCE}" (at 0 0) (layer "F.Fab") hide
-      (effects (font (size 1 1) (thickness 0.15)))
-    )
-    (fp_line (start -0.63 -1.27) (end -0.63 1.27) (layer "F.CrtYd") (width 0.05))
-    (fp_line (start -0.63 1.27) (end 0.63 1.27) (layer "F.CrtYd") (width 0.05))
-    (fp_line (start 0.63 1.27) (end 0.63 -1.27) (layer "F.CrtYd") (width 0.05))
-    (fp_line (start 0.63 -1.27) (end -0.63 -1.27) (layer "F.CrtYd") (width 0.05))
-    (fp_line (start -0.63 1.27) (end -0.63 -1.27) (layer "F.Fab") (width 0.1))
-    (fp_line (start 0.63 1.27) (end -0.63 1.27) (layer "F.Fab") (width 0.1))
-    (fp_line (start 0.63 -1.27) (end 0.63 1.27) (layer "F.Fab") (width 0.1))
-    (fp_line (start -0.63 -1.27) (end 0.63 -1.27) (layer "F.Fab") (width 0.1))
-    (pad "" smd roundrect (at 0 0) (size 1 2) (layers "B.Cu" "B.Paste" "B.Mask") (roundrect_rratio 0.25)
-      (net 1 "GND"))
-  )
   (footprint "Connector_PinHeader_2.54mm:PinHeader_1x03_P2.54mm_Vertical" (layer "F.Cu")
     (at 78.105 129.525 180)
@@
       (rotate (xyz 0 0 0))
     )
-  )
-  (footprint "" (layer "F.Cu")
-    (at 112.395 55.245)
-    (fp_text reference "" (at 0 0) (layer "F.SilkS")
-      (effects (font (size 1.27 1.27) (thickness 0.15)))
-    )
-    (fp_text value "" (at 0 0) (layer "F.SilkS")
-      (effects (font (size 1.27 1.27) (thickness 0.15)))
-    )
-    (pad "" smd roundrect (at 0 0) (size 1 2) (layers "B.Cu" "B.Paste" "B.Mask") (roundrect_rratio 0.25)
-      (net 1 "GND"))
-  )
-  (footprint "" (layer "F.Cu")
-    (at 74.93 71.12)
-    (fp_text reference "" (at 0 0) (layer "F.SilkS")
-      (effects (font (size 1.27 1.27) (thickness 0.15)))
-    )
-    (fp_text value "" (at 0 0) (layer "F.SilkS")
-      (effects (font (size 1.27 1.27) (thickness 0.15)))
-    )
-    (pad "" smd roundrect (at 0 0) (size 1 2) (layers "B.Cu" "B.Paste" "B.Mask") (roundrect_rratio 0.25)
-      (net 1 "GND"))
   )
   (footprint "Connector_Coaxial:SMA_Samtec_SMA-J-P-X-ST-EM1_EdgeMount" (layer "F.Cu")
@@
     )
   )
-  (footprint "Connector_Wire:SolderWirePad_1x01_SMD_1x2mm" (layer "F.Cu")
-    (at 74.93 55.245)
-    (descr "Wire Pad, Square, SMD Pad,  1mm x 2mm,")
-    (tags "MesurementPoint Square SMDPad 1mmx2mm ")
-    (attr exclude_from_pos_files exclude_from_bom)
-    (fp_text reference "REF**" (at 0 -2.54) (layer "F.SilkS") hide
-      (effects (font (size 1 1) (thickness 0.15)))
-    )
-    (fp_text value "SolderWirePad_1x01_SMD_1x2mm" (at 0 2.54) (layer "F.Fab") hide
-      (effects (font (size 1 1) (thickness 0.15)))
-    )
-    (fp_text user "${REFERENCE}" (at 0 0) (layer "F.Fab") hide
-      (effects (font (size 1 1) (thickness 0.15)))
-    )
-    (fp_line (start 0.63 -1.27) (end -0.63 -1.27) (layer "F.CrtYd") (width 0.05))
-    (fp_line (start -0.63 -1.27) (end -0.63 1.27) (layer "F.CrtYd") (width 0.05))
-    (fp_line (start 0.63 1.27) (end 0.63 -1.27) (layer "F.CrtYd") (width 0.05))
-    (fp_line (start -0.63 1.27) (end 0.63 1.27) (layer "F.CrtYd") (width 0.05))
-    (fp_line (start 0.63 -1.27) (end 0.63 1.27) (layer "F.Fab") (width 0.1))
-    (fp_line (start 0.63 1.27) (end -0.63 1.27) (layer "F.Fab") (width 0.1))
-    (fp_line (start -0.63 1.27) (end -0.63 -1.27) (layer "F.Fab") (width 0.1))
-    (fp_line (start -0.63 -1.27) (end 0.63 -1.27) (layer "F.Fab") (width 0.1))
-    (pad "" smd roundrect (at 0 0) (size 1 2) (layers "B.Cu" "B.Paste" "B.Mask") (roundrect_rratio 0.25)
-      (net 1 "GND"))
-  )
   (footprint "lora_tracker:ATGM336H" (layer "F.Cu")
     (at 97.79 89.535)
@@
     (fp_line (start -2.54 0.32) (end -1.59 1.27) (layer "B.Fab") (width 0.1))
     (pad "1" smd rect (at -2.525 0) (size 3.15 1) (layers "B.Cu" "B.Paste" "B.Mask")
-      (net 39 "Net-(U5-Pad9)") (pinfunction "Pin_1") (pintype "passive"))
+      (net 39 "Net-(J2-Pad1)") (pinfunction "Pin_1") (pintype "passive"))
     (pad "2" smd rect (at 2.525 0) (size 3.15 1) (layers "B.Cu" "B.Paste" "B.Mask")
-      (net 40 "Net-(U5-Pad8)") (pinfunction "Pin_2") (pintype "passive"))
+      (net 40 "Net-(J2-Pad2)") (pinfunction "Pin_2") (pintype "passive"))
     (model "${KICAD6_3DMODEL_DIR}/Connector_PinHeader_2.54mm.3dshapes/PinHeader_2x01_P2.54mm_Vertical_SMD.wrl"
       (offset (xyz 0 0 0))

Commit message: Update schematics
Routing:
- net GND: vias 152 -> 154
Changed lines of the file:
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@@
   (via (at 91.44 63.5) (size 0.8) (drill 0.4) (layers "F.Cu" "B.Cu") (free) (net 1))
   (via (at 112.395 77.47) (size 0.8) (drill 0.4) (layers "F.Cu" "B.Cu") (net 1))
+  (via (at 112.395 71.755) (size 0.8) (drill 0.4) (layers "F.Cu" "B.Cu") (free) (net 1))
   (via (at 103.505 50.165) (size 0.8) (drill 0.4) (layers "F.Cu" "B.Cu") (net 1))
   (via (at 104.775 63.5) (size 0.8) (drill 0.4) (layers "F.Cu" "B.Cu") (free) (net 1))
   (via (at 92.71 81.28) (size 0.8) (drill 0.4) (layers "F.Cu" "B.Cu") (free) (net 1))
-  (via (at 98.425 89.535) (size 0.8) (drill 0.4) (layers "F.Cu" "B.Cu") (free) (net 1))
+  (via (at 99.06 90.17) (size 0.8) (drill 0.4) (layers "F.Cu" "B.Cu") (free) (net 1))
   (via (at 93.98 68.58) (size 0.8) (drill 0.4) (layers "F.Cu" "B.Cu") (free) (net 1))
   (via (at 80.01 60.325) (size 0.8) (drill 0.4) (layers "F.Cu" "B.Cu") (free) (net 1))
   (via (at 80.01 73.66) (size 0.8) (drill 0.4) (layers "F.Cu" "B.Cu") (free) (net 1))
-  (via (at 74.93 73.152) (size 0.8) (drill 0.4) (layers "F.Cu" "B.Cu") (net 1))
+  (via (at 74.93 74.295) (size 0.8) (drill 0.4) (layers "F.Cu" "B.Cu") (net 1))
   (via (at 112.395 109.728) (size 0.8) (drill 0.4) (layers "F.Cu" "B.Cu") (net 1))
   (via (at 88.265 67.31) (size 0.8) (drill 0.4) (layers "F.Cu" "B.Cu") (free) (net 1))
-  (via (at 100.965 47.625) (size 0.8) (drill 0.4) (layers "F.Cu" "B.Cu") (net 1))
   (via (at 100.965 67.31) (size 0.8) (drill 0.4) (layers "F.Cu" "B.Cu") (free) (net 1))
   (via (at 108.585 94.615) (size 0.8) (drill 0.4) (layers "F.Cu" "B.Cu") (free) (net 1))
@@
   (via (at 104.14 127) (size 0.8) (drill 0.4) (layers "F.Cu" "B.Cu") (free) (net 1))
   (via (at 87.63 74.93) (size 0.8) (drill 0.4) (layers "F.Cu" "B.Cu") (free) (net 1))
+  (via (at 86.995 53.34) (size 0.8) (drill 0.4) (layers "F.Cu" "B.Cu") (net 1))
   (via (at 87.884 44.45) (size 0.8) (drill 0.4) (layers "F.Cu" "B.Cu") (net 1))
   (via (at 112.395 130.048) (size 0.8) (drill 0.4) (layers "F.Cu" "B.Cu") (net 1))
@@
   (via (at 90.17 131.445) (size 0.8) (drill 0.4) (layers "F.Cu" "B.Cu") (free) (net 1))
   (via (at 93.98 71.12) (size 0.8) (drill 0.4) (layers "F.Cu" "B.Cu") (free) (net 1))
+  (via (at 112.395 55.88) (size 0.8) (drill 0.4) (layers "F.Cu" "B.Cu") (net 1))
   (via (at 80.645 91.44) (size 0.8) (drill 0.4) (layers "F.Cu" "B.Cu") (free) (net 1))
   (via (at 106.045 81.915) (size 0.8) (drill 0.4) (layers "F.Cu" "B.Cu") (net 1))
@@
   (via (at 104.14 73.66) (size 0.8) (drill 0.4) (layers "F.Cu" "B.Cu") (net 1))
   (via (at 95.885 123.825) (size 0.8) (drill 0.4) (layers "F.Cu" "B.Cu") (free) (net 1))
-  (via (at 101.6 81.915) (size 0.8) (drill 0.4) (layers "F.Cu" "B.Cu") (free) (net 1))
+  (via (at 101.6 82.55) (size 0.8) (drill 0.4) (layers "F.Cu" "B.Cu") (free) (net 1))
   (via (at 95.25 60.96) (size 0.8) (drill 0.4) (layers "F.Cu" "B.Cu") (free) (net 1))
+  (via (at 112.395 69.215) (size 0.8) (drill 0.4) (layers "F.Cu" "B.Cu") (free) (net 1))
   (via (at 78.74 57.15) (size 0.8) (drill 0.4) (layers "F.Cu" "B.Cu") (net 1))
   (via (at 109.855 69.215) (size 0.8) (drill 0.4) (layers "F.Cu" "B.Cu") (free) (net 1))
@@
   (via (at 108.585 102.235) (size 0.8) (drill 0.4) (layers "F.Cu" "B.Cu") (free) (net 1))
   (via (at 110.49 83.82) (size 0.8) (drill 0.4) (layers "F.Cu" "B.Cu") (net 1))
-  (via (at 74.93 52.832) (size 0.8) (drill 0.4) (layers "F.Cu" "B.Cu") (net 1))
+  (via (at 74.93 53.975) (size 0.8) (drill 0.4) (layers "F.Cu" "B.Cu") (net 1))
   (via (at 85.725 120.015) (size 0.8) (drill 0.4) (layers "F.Cu" "B.Cu") (free) (net 1))
   (via (at 111.125 45.72) (size 4) (drill 2.7) (layers "F.Cu" "B.Cu") (free) (net 1))
@@
   (via (at 99.06 94.615) (size 0.8) (drill 0.4) (layers "F.Cu" "B.Cu") (free) (net 1))
   (via (at 106.045 73.66) (size 0.8) (drill 0.4) (layers "F.Cu" "B.Cu") (free) (net 1))
-  (via (at 74.93 75.184) (size 0.8) (drill 0.4) (layers "F.Cu" "B.Cu") (net 1))
   (via (at 112.395 52.705) (size 0.8) (drill 0.4) (layers "F.Cu" "B.Cu") (net 1))
   (via (at 83.82 84.455) (size 0.8) (drill 0.4) (layers "F.Cu" "B.Cu") (free) (net 1))
   (via (at 112.395 113.792) (size 0.8) (drill 0.4) (layers "F.Cu" "B.Cu") (net 1))
   (via (at 102.87 113.665) (size 0.8) (drill 0.4) (layers "F.Cu" "B.Cu") (free) (net 1))
-  (via (at 109.855 72.39) (size 0.8) (drill 0.4) (layers "F.Cu" "B.Cu") (free) (net 1))
+  (via (at 109.855 71.755) (size 0.8) (drill 0.4) (layers "F.Cu" "B.Cu") (free) (net 1))
   (via (at 97.79 108.585) (size 0.8) (drill 0.4) (layers "F.Cu" "B.Cu") (free) (net 1))
   (via (at 74.93 50.165) (size 0.8) (drill 0.4) (layers "F.Cu" "B.Cu") (net 1))
@@
   (via (at 106.045 80.01) (size 0.8) (drill 0.4) (layers "F.Cu" "B.Cu") (free) (net 1))
   (via (at 93.345 104.775) (size 0.8) (drill 0.4) (layers "F.Cu" "B.Cu") (free) (net 1))
-  (via (at 109.22 57.15) (size 0.8) (drill 0.4) (layers "F.Cu" "B.Cu") (free) (net 1))
+  (via (at 108.585 57.785) (size 0.8) (drill 0.4) (layers "F.Cu" "B.Cu") (free) (net 1))
   (via (at 112.395 93.472) (size 0.8) (drill 0.4) (layers "F.Cu" "B.Cu") (net 1))
   (via (at 83.82 104.14) (size 0.8) (drill 0.4) (layers "F.Cu" "B.Cu") (free) (net 1))
   (via (at 84.455 49.53) (size 0.8) (drill 0.4) (layers "F.Cu" "B.Cu") (net 1))
   (via (at 95.885 67.945) (size 0.8) (drill 0.4) (layers "F.Cu" "B.Cu") (free) (net 1))
-  (via (at 110.49 74.295) (size 0.8) (drill 0.4) (layers "F.Cu" "B.Cu") (net 1))
+  (via (at 109.855 74.295) (size 0.8) (drill 0.4) (layers "F.Cu" "B.Cu") (net 1))
   (via (at 94.615 114.3) (size 0.8) (drill 0.4) (layers "F.Cu" "B.Cu") (free) (net 1))
   (via (at 108.585 117.475) (size 0.8) (drill 0.4) (layers "F.Cu" "B.Cu") (free) (net 1))

Commit message: Update schematics
Parts:
- added J3: Conn_01x01, TestPoint:TestPoint_Pad_1.5x1.5mm, B.Cu at (74.9, 71.1)
- added J5: Conn_01x01, TestPoint:TestPoint_Pad_1.5x1.5mm, B.Cu at (74.9, 55.2)
- added J6: Conn_01x01, TestPoint:TestPoint_Pad_1.5x1.5mm, B.Cu at (112.4, 55.2)
- added J7: Conn_01x01, TestPoint:TestPoint_Pad_1.5x1.5mm, B.Cu at (112.4, 71.1)
- R2: value 1k -> 10k
Connections:
- SW1 pad : GND -> (no net)
Routing:
- net GND: vias 154 -> 149

Commit message: Update schematics
Other:
- rule pad_to_mask_clearance: 0.051 -> 0
