File: extras/schematics/lora_tracker.kicad_sch (KiCad schematic)
At the start: 18 parts, among them J1 Conn_Coaxial, J2 Conn_01x10_Female, J3 Conn_01x12_Female, J4 Conn_01x03_Female, U1 ESP32, U2 E22-400M30S, U3 Ai-Thinker-Ra-01

Commit message: Updates
Parts:
- removed JP1, JP2, JP3: SolderJumper_3_Open, Jumper:SolderJumper-3_P1.3mm_Open_Pad1.0x1.5mm, symbol lora_tracker-rescue:SolderJumper_3_Open-Jumper
- removed JP4, JP5, JP6, JP7, JP8: SolderJumper_2_Open, Jumper:SolderJumper-2_P1.3mm_Open_Pad1.0x1.5mm, symbol Jumper:SolderJumper_2_Open
- removed U1: ESP32, lora_tracker:esp32-devkit-wide, symbol lora_tracker:ESP32
- added U1: ESP32_30pin, lora_tracker:esp32-devkit-wide_copy, symbol lora_tracker:ESP32_30pin
- C1, C3: footprint Capacitor_SMD:C_0603_1608Metric_Pad1.05x0.95mm_HandSolder -> Capacitor_SMD:C_0603_1608Metric_Pad1.08x0.95mm_HandSolder
- J1: footprint Connector_Coaxial:SMA_Samtec_SMA-J-P-H-ST-EM1_EdgeMount -> Connector_Coaxial:SMA_Samtec_SMA-J-P-X-ST-EM1_EdgeMount
Connections:
- net 3v3: now also U1.16 (3V3)
- net BUSY: now also U1.11 (GPIO14)
- net DIO1: now also U1.12 (GPIO12)
- net EN: now also U1.1 (EN)
- net GND: now also U1.14 (GND), U1.17 (GND)
- net GPIO1: now also U1.28 (TX0/01)
- net GPIO13: now also U1.13 (GPIO13)
- net GPIO15: now also U1.18 (GPIO15)
- net GPIO16: now also U1.21 (RX2/16)
- net GPIO17: now also U1.22 (TX2/17)
- net GPIO2: now also U1.19 (GPIO2)
- net GPIO21: now also U1.26 (GPIO21)
- net GPIO22: now also U1.29 (GPIO22)
- net GPIO25: now also U1.8 (GPIO25)
- net GPIO26: now also U1.9 (GPIO26)
- net GPIO3: now also U1.27 (RX0/03)
- net GPIO34: now also U1.4 (GPIO34)
- net GPIO35: now also U1.5 (GPIO35)
- net GPIO36: now also U1.2 (VP/36)
- net GPIO39: now also U1.3 (VN/39)
- net GPIO4: now also U1.20 (GPIO4)
- net MISO: now also U1.25 (GPIO19)
- net MOSI: now also U1.30 (GPIO23)
- net NRST: now also U1.10 (GPIO27)
- net NSS: now also U1.23 (GPIO5)
- net RXEN: now also U1.6 (GPIO32)
- net SCK: now also U1.24 (GPIO18)
- net TXEN: now also U1.7 (GPIO33)
- net VCC: now also U1.15 (VIN)
- net GPIO0: no longer names the net of J3.5 (Pin_5)
- net GPIO10: no longer names the net of J2.1 (Pin_1)
- net GPIO7: no longer names the net of J3.1 (Pin_1)
- net GPIO8: no longer names the net of J3.2 (Pin_2)
- net GPIO9: no longer names the net of J2.2 (Pin_2)
- no-connect marks 5 -> 10
Other:
- note removed: "ESP32 SPI flavours"
- note removed: "ESP32 options"
- moved on the sheet: C1, C2, C3, J1, J2, J3, J4, U2, U3

Commit message: Update schematics
Parts:
- removed J2: Conn_01x10_Female, Connector_PinSocket_2.54mm:PinSocket_1x10_P2.54mm_Vertical, symbol Connector:Conn_01x10_Female
- removed J3: Conn_01x12_Female, Connector_PinSocket_2.54mm:PinSocket_1x12_P2.54mm_Vertical, symbol Connector:Conn_01x12_Female
- added C4, C5, C6, C7: 100nF, Capacitor_SMD:C_0603_1608Metric_Pad1.08x0.95mm_HandSolder, symbol Device:C
- added C8: 0.1uF, symbol Device:C
- added R1: 100k, symbol Device:R
- added R2: 1k, symbol Device:R
- added SW1: SW_Push, symbol Switch:SW_Push
- added U4: INP441, symbol lora_tracker:INP441
- added U5: MAX98357A, symbol lora_tracker:MAX98357A
- added U6: SSD1306, symbol lora_tracker:SSD1306
- added U7: KY040, symbol lora_tracker:KY040
- J1: value Conn_Coaxial -> Coax
- J4: value Conn_01x03_Female -> Pwr
- U1: value ESP32_30pin -> ESP32
- U3: value Ai-Thinker-Ra-01 -> RA-01
Connections:
- net GPIO2 is gone; now on net 3v3: U1.19 (GPIO2)
- net 3v3: now also C4.1, C5.1, R2.1, U4.4 (SD), U4.5 (VDD), U7.5 (VCC)
- net GND: now also C4.2, C5.2, C6.2, C7.2, C8.2, R1.2, SW1.2, U4.1 (L/R), U4.6 (GND), U5.6 (GND), U6.4 (GND), U7.1 (GND)
- net GPIO13: now also U5.1 (LRC)
- net GPIO15: now also U4.2 (WS)
- net GPIO16: now also U7.3 (S2)
- net GPIO17: now also U7.2 (S1)
- net GPIO21: now also U6.1 (SDA)
- net GPIO22: now also U6.2 (SCL)
- net GPIO25: now also U5.3 (DIN)
- net GPIO26: now also U5.2 (BCLK)
- net GPIO34: now also U7.4 (KEY)
- net GPIO39: now also C8.1, R2.2, SW1.1
- net GPIO4: now also U4.3 (SCK)
- net ANT: now reaches J1.1 (In), U2.21 (ANT), U3.1 (Ant)
- net VCC renamed 5V
- net 5V: now also C6.1, C7.1, U5.5 (SD), U5.7 (VIN), U6.3 (VCC)
- new net: R1.1, U5.4 (GAIN)
- no-connect marks 10 -> 5
Other:
- moved on the sheet: C3

Commit message: Update schematics
Parts:
- C8: footprint (none) -> Capacitor_SMD:C_0603_1608Metric_Pad1.08x0.95mm_HandSolder
- R1, R2: footprint (none) -> Resistor_SMD:R_0603_1608Metric_Pad0.98x0.95mm_HandSolder
- SW1: footprint (none) -> Button_Switch_THT:SW_Tactile_SKHH_Angled
Other:
- moved on the sheet: C1, C2

Commit message: Updated schematics
Parts:
- removed U7: KY040, symbol lora_tracker:KY040
- added C9: 47uF, Capacitor_THT:CP_Radial_D4.0mm_P2.00mm, symbol Device:C_Polarized
- added R3, R4, R5: 10k, Resistor_SMD:R_0603_1608Metric_Pad0.98x0.95mm_HandSolder, symbol Device:R
- added U7: EC11, lora_tracker:ec11, symbol lora_tracker:EC11
- J1: value Coax -> ANT
- U1: footprint lora_tracker:esp32-devkit-wide_copy -> lora_tracker:esp32-devkit-wide_30pin
- U4: footprint (none) -> lora_tracker:inp441
- U5: footprint (none) -> lora_tracker:MAX98357A
- U6: footprint (none) -> lora_tracker:SSD1306
Connections:
- net 3v3: now also R3.1, R4.1, R5.1; no longer U1.19 (GPIO2), U4.4 (SD)
- net 5V: now also C9.1
- net GND: now also C9.2, U7.C (GND), U7.MP, U7.S1 (GND)
- net GPIO16: now also R3.2, U7.B (OUTB)
- net GPIO17: now also R4.2, U7.A (OUTA)
- net GPIO34: now also R5.2, U7.S2 (SWITCH)
- new net GPIO2: U1.19 (GPIO2), U4.4 (SD)
Other:
- moved on the sheet: C8, J1, R2, SW1

Commit message: Update schematics
Parts:
- added R6, R7: 10k, Resistor_SMD:R_0603_1608Metric_Pad0.98x0.95mm_HandSolder, symbol Device:R
- J4: value Pwr -> Conn_01x03_Female; footprint Connector_PinSocket_2.54mm:PinSocket_1x03_P2.54mm_Vertical -> Connector_PinHeader_2.54mm:PinHeader_1x03_P2.54mm_Vertical
Connections:
- net 3v3: no longer J4.2 (Pin_2)
- net 5V: now also J4.2 (Pin_2); no longer J4.3 (Pin_3)
- net GND: now also R7.2
- net GPIO36: now also R6.2, R7.1
- new net: J4.3 (Pin_3), R6.1
Other:
- moved on the sheet: C1, C2, C3, U3

Commit message: Update schematics
Parts:
- added C10: 100nF, Capacitor_SMD:C_0603_1608Metric_Pad1.08x0.95mm_HandSolder, symbol Device:C
Connections:
- net GND: now also C10.2
- net GPIO36: now also C10.1
Changed lines of the file:
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@@
 (kicad_sch (version 20211123) (generator eeschema)
   (paper "A4")
+  (junction (at 124.46 30.48) (diameter 0) (color 0 0 0 0)
+  )
   (junction (at 194.31 81.28) (diameter 0) (color 0 0 0 0)
   )
@@
     (stroke (width 0) (type default) (color 0 0 0 0))
   )
-  (wire (pts (xy 114.3 30.48) (xy 123.19 30.48))
+  (wire (pts (xy 114.3 30.48) (xy 124.46 30.48))
     (stroke (width 0) (type default) (color 0 0 0 0))
   )
@@
     (stroke (width 0) (type default) (color 0 0 0 0))
   )
+  (wire (pts (xy 124.46 39.37) (xy 124.46 43.18))
+    (stroke (width 0) (type default) (color 0 0 0 0))
+  )
   (wire (pts (xy 26.67 29.21) (xy 31.75 29.21))
     (stroke (width 0) (type default) (color 0 0 0 0))
@@
     (stroke (width 0) (type default) (color 0 0 0 0))
   )
+  (wire (pts (xy 124.46 30.48) (xy 124.46 31.75))
+    (stroke (width 0) (type default) (color 0 0 0 0))
+  )
   (wire (pts (xy 82.55 160.02) (xy 82.55 167.64))
+    (stroke (width 0) (type default) (color 0 0 0 0))
+  )
+  (wire (pts (xy 124.46 30.48) (xy 130.81 30.48))
     (stroke (width 0) (type default) (color 0 0 0 0))
   )
@@
     )
   )
-  (global_label "GPIO36" (shape input) (at 123.19 30.48 0) (fields_autoplaced)
-    (effects (font (size 1.27 1.27)) (justify left))
-    (property "Intersheet References" "${INTERSHEET_REFS}" (id 0) (at 132.4085 30.4006 0)
+  (global_label "GPIO36" (shape input) (at 130.81 30.48 0) (fields_autoplaced)
+    (effects (font (size 1.27 1.27)) (justify left))
+    (property "Intersheet References" "${INTERSHEET_REFS}" (id 0) (at 140.0285 30.4006 0)
       (effects (font (size 1.27 1.27)) (justify left) hide)
     )
@@
     (effects (font (size 1.27 1.27)) (justify left))
     (property "Intersheet References" "${INTERSHEET_REFS}" (id 0) (at -25.4 -35.56 0)
+      (effects (font (size 1.27 1.27)) hide)
+    )
+  )
+  (global_label "GND" (shape input) (at 124.46 43.18 270) (fields_autoplaced)
+    (effects (font (size 1.27 1.27)) (justify right))
+    (property "Intersheet References" "${INTERSHEET_REFS}" (id 0) (at 275.59 -163.83 0)
       (effects (font (size 1.27 1.27)) hide)
     )
@@
     (pin "4-UD")
   )
+  (symbol (lib_id "Device:C") (at 124.46 35.56 0) (unit 1)
+    (in_bom yes) (on_board yes)
+    (property "Reference" "C10" (id 0) (at 127.381 34.3916 0)
+      (effects (font (size 1.27 1.27)) (justify left))
+    )
+    (property "Value" "100nF" (id 1) (at 127.381 36.703 0)
+      (effects (font (size 1.27 1.27)) (justify left))
+    )
+    (property "Footprint" "Capacitor_SMD:C_0603_1608Metric_Pad1.08x0.95mm_HandSolder" (id 2) (at 125.4252 39.37 0)
+      (effects (font (size 1.27 1.27)) hide)
+    )
+    (property "Datasheet" "~" (id 3) (at 124.46 35.56 0)
+      (effects (font (size 1.27 1.27)) hide)
+    )
+    (pin "1")
+    (pin "2")
+  )
   (symbol (lib_id "Device:R") (at 90.17 156.21 0) (unit 1)
     (in_bom yes) (on_board yes) (fields_autoplaced)
@@
       (reference "C9") (unit 1) (value "47uF") (footprint "Capacitor_THT:CP_Radial_D4.0mm_P2.00mm")
     )
+    (path "/f0bcdabe-6864-48d2-bcb4-aae285e928df"
+      (reference "C10") (unit 1) (value "100nF") (footprint "Capacitor_SMD:C_0603_1608Metric_Pad1.08x0.95mm_HandSolder")
+    )
     (path "/c5fb8d0b-52b5-449b-965e-53dc20584b98"

Commit message: Update schematics
Connections:
- net EN: no longer names the net of U1.1 (EN)
- net GPIO1: no longer names the net of U1.28 (TX0/01)
- net GPIO3: no longer names the net of U1.27 (RX0/03)
- net GPIO35: no longer names the net of U1.5 (GPIO35)
- no-connect marks 5 -> 9
Changed lines of the file:
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@@
   )
   (no_connect (at 205.74 71.12))
+  (no_connect (at 60.96 29.21))
   (no_connect (at 175.26 54.61))
+  (no_connect (at 60.96 26.67))
+  (no_connect (at 26.67 31.75))
+  (no_connect (at 26.67 21.59))
   (no_connect (at 175.26 52.07))
   (no_connect (at 175.26 49.53))
@@
     )
   )
+  (global_label "GPIO21" (shape input) (at 60.96 31.75 0) (fields_autoplaced)
+    (effects (font (size 1.27 1.27)) (justify left))
+    (property "Intersheet References" "${INTERSHEET_REFS}" (id 0) (at 70.1785 31.6706 0)
+      (effects (font (size 1.27 1.27)) (justify left) hide)
+    )
+  )
   (global_label "DIO1" (shape input) (at 259.08 81.28 0) (fields_autoplaced)
     (effects (font (size 1.27 1.27)) (justify left))
@@
     (property "Intersheet References" "${INTERSHEET_REFS}" (id 0) (at 118.11 182.88 0)
       (effects (font (size 1.27 1.27)) hide)
+    )
+  )
+  (global_label "GPIO2" (shape input) (at 60.96 49.53 0) (fields_autoplaced)
+    (effects (font (size 1.27 1.27)) (justify left))
+    (property "Intersheet References" "${INTERSHEET_REFS}" (id 0) (at 68.969 49.4506 0)
+      (effects (font (size 1.27 1.27)) (justify left) hide)
     )
   )
@@
     )
   )
-  (global_label "EN" (shape input) (at 26.67 21.59 180) (fields_autoplaced)
-    (effects (font (size 1.27 1.27)) (justify right))
-    (property "Intersheet References" "${INTERSHEET_REFS}" (id 0) (at -25.4 -30.48 0)
-      (effects (font (size 1.27 1.27)) hide)
-    )
-  )
   (global_label "GPIO16" (shape input) (at 74.93 167.64 180) (fields_autoplaced)
     (effects (font (size 1.27 1.27)) (justify right))
@@
     )
   )
-  (global_label "GPIO15" (shape input) (at 60.96 52.07 0) (fields_autoplaced)
-    (effects (font (size 1.27 1.27)) (justify left))
-    (property "Intersheet References" "${INTERSHEET_REFS}" (id 0) (at -25.4 -35.56 0)
-      (effects (font (size 1.27 1.27)) hide)
-    )
-  )
   (global_label "GND" (shape input) (at 124.46 43.18 270) (fields_autoplaced)
     (effects (font (size 1.27 1.27)) (justify right))
@@
     )
   )
+  (global_label "GPIO4" (shape input) (at 60.96 46.99 0) (fields_autoplaced)
+    (effects (font (size 1.27 1.27)) (justify left))
+    (property "Intersheet References" "${INTERSHEET_REFS}" (id 0) (at 68.969 46.9106 0)
+      (effects (font (size 1.27 1.27)) (justify left) hide)
+    )
+  )
   (global_label "MISO" (shape input) (at 259.08 66.04 0) (fields_autoplaced)
     (effects (font (size 1.27 1.27)) (justify left))
@@
     )
   )
-  (global_label "GPIO3" (shape input) (at 60.96 29.21 0) (fields_autoplaced)
-    (effects (font (size 1.27 1.27)) (justify left))
-    (property "Intersheet References" "${INTERSHEET_REFS}" (id 0) (at -25.4 -30.48 0)
-      (effects (font (size 1.27 1.27)) hide)
-    )
-  )
   (global_label "GND" (shape input) (at 143.51 113.03 270) (fields_autoplaced)
     (effects (font (size 1.27 1.27)) (justify right))
@@
     )
   )
-  (global_label "GPIO35" (shape input) (at 26.67 31.75 180) (fields_autoplaced)
-    (effects (font (size 1.27 1.27)) (justify right))
-    (property "Intersheet References" "${INTERSHEET_REFS}" (id 0) (at -25.4 -30.48 0)
-      (effects (font (size 1.27 1.27)) hide)
-    )
-  )
   (global_label "MOSI" (shape input) (at 60.96 21.59 0) (fields_autoplaced)
-    (effects (font (size 1.27 1.27)) (justify left))
-    (property "Intersheet References" "${INTERSHEET_REFS}" (id 0) (at -25.4 -30.48 0)
-      (effects (font (size 1.27 1.27)) hide)
-    )
-  )
-  (global_label "GPIO2" (shape input) (at 60.96 49.53 0) (fields_autoplaced)
-    (effects (font (size 1.27 1.27)) (justify left))
-    (property "Intersheet References" "${INTERSHEET_REFS}" (id 0) (at -25.4 -35.56 0)
-      (effects (font (size 1.27 1.27)) hide)
-    )
-  )
-  (global_label "GPIO1" (shape input) (at 60.96 26.67 0) (fields_autoplaced)
     (effects (font (size 1.27 1.27)) (justify left))
     (property "Intersheet References" "${INTERSHEET_REFS}" (id 0) (at -25.4 -30.48 0)
@@
     )
   )
-  (global_label "GPIO4" (shape input) (at 60.96 46.99 0) (fields_autoplaced)
-    (effects (font (size 1.27 1.27)) (justify left))
-    (property "Intersheet References" "${INTERSHEET_REFS}" (id 0) (at -25.4 -33.02 0)
-      (effects (font (size 1.27 1.27)) hide)
-    )
-  )
   (global_label "MISO" (shape input) (at 147.32 54.61 180) (fields_autoplaced)
     (effects (font (size 1.27 1.27)) (justify right))
@@
   (global_label "GND" (shape input) (at 102.87 27.94 0) (fields_autoplaced)
     (effects (font (size 1.27 1.27)) (justify left))
-    (property "Intersheet References" "${INTERSHEET_REFS}" (id 0) (at -104.14 -123.19 0)
-      (effects (font (size 1.27 1.27)) hide)
-    )
-  )
-  (global_label "GPIO21" (shape input) (at 60.96 31.75 0) (fields_autoplaced)
-    (effects (font (size 1.27 1.27)) (justify left))
-    (property "Intersheet References" "${INTERSHEET_REFS}" (id 0) (at -25.4 -30.48 0)
-      (effects (font (size 1.27 1.27)) hide)
+    (property "Intersheet References" "${INTERSHEET_REFS}" (id 0) (at 109.0647 27.8606 0)
+      (effects (font (size 1.27 1.27)) (justify left) hide)
     )
   )
@@
     )
   )
+  (global_label "GPIO15" (shape input) (at 60.96 52.07 0) (fields_autoplaced)
+    (effects (font (size 1.27 1.27)) (justify left))
+    (property "Intersheet References" "${INTERSHEET_REFS}" (id 0) (at 70.1785 51.9906 0)
+      (effects (font (size 1.27 1.27)) (justify left) hide)
+    )
+  )
