File: extras/schematics/lora_tracker.kicad_sch (KiCad schematic)
At the start: 27 parts, among them J1 ANT, J4 Conn_01x03_Female, SW1 SW_Push, U1 ESP32, U2 E22-400M30S, U3 RA-01, U4 INP441, U5 MAX98357A, U6 SSD1306, U7 EC11

Commit message: Update schematics
Parts:
- renumbered U7 to SW2
Changed lines of the file:
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@@
   (symbol (lib_id "lora_tracker:EC11") (at 105.41 161.29 0) (unit 1)
     (in_bom yes) (on_board yes) (fields_autoplaced)
-    (property "Reference" "U7" (id 0) (at 105.41 160.181 0))
+    (property "Reference" "SW2" (id 0) (at 105.41 160.181 0))
     (property "Value" "EC11" (id 1) (at 105.41 162.7179 0))
     (property "Footprint" "lora_tracker:ec11" (id 2) (at 105.41 161.29 0)
@@
       (reference "SW1") (unit 1) (value "SW_Push") (footprint "Button_Switch_THT:SW_Tactile_SKHH_Angled")
     )
+    (path "/be6a4cbb-024a-479b-93d8-f83ffb72c45d"
+      (reference "SW2") (unit 1) (value "EC11") (footprint "lora_tracker:ec11")
+    )
     (path "/60d2b1ac-2da1-41aa-ada2-be6b13794aa0"
       (reference "U1") (unit 1) (value "ESP32") (footprint "lora_tracker:esp32-devkit-wide_30pin")
@@
       (reference "U6") (unit 1) (value "SSD1306") (footprint "lora_tracker:SSD1306")
     )
-    (path "/be6a4cbb-024a-479b-93d8-f83ffb72c45d"
-      (reference "U7") (unit 1) (value "EC11") (footprint "lora_tracker:ec11")
-    )
-  )
+  )

Commit message: Update schematics
Parts:
- added U7: ATGM336H, symbol lora_tracker:ATGM336H
Connections:
- net 3v3: now also U7.5 (VCC); no longer C4.1
- net GND: now also U7.4 (GND)
- net GPIO2: now also C4.1
- net GPIO3: now reaches U1.27 (RX0/03)
- net GPIO3: now also U7.3 (TX)
- net GPIO1: now reaches U1.28 (TX0/01)
- net GPIO1: now also U7.2 (RX)
- no-connect marks 9 -> 8
Other:
- note added: "Antenna connection"
- note added: "Audio i2s amplifier"
- note added: "ESP32 MCU"
- note added: "GPS module"
- note added: "Microphone i2s"
- note added: "PTT button"
- note added: "Power input and battery monitor"
- note added: "Radio modules"
- note added: "Rotary encoder with button"
- note added: "Screen"
- moved on the sheet: C1, C10, C2, C3, C4, C5, C6, C7, C8, C9, J1, J4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

Commit message: Update schematics
Parts:
- added C11: 100nF, Capacitor_SMD:C_0603_1608Metric_Pad1.08x0.95mm_HandSolder, symbol Device:C
- U7: footprint (none) -> lora_tracker:ATGM336H
Connections:
- net 3v3: now also C4.1, C11.1
- net GND: now also C11.2
- net GPIO2: no longer C4.1
Changed lines of the file:
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@@
   (junction (at 118.11 34.29) (diameter 0) (color 0 0 0 0)
   )
+  (junction (at 149.86 83.82) (diameter 0) (color 0 0 0 0)
+  )
   (junction (at 44.45 151.13) (diameter 0) (color 0 0 0 0)
   )
@@
   (junction (at 193.04 115.57) (diameter 0) (color 0 0 0 0)
   )
-  (junction (at 46.99 115.57) (diameter 0) (color 0 0 0 0)
+  (junction (at 46.99 111.76) (diameter 0) (color 0 0 0 0)
   )
   (junction (at 102.87 29.21) (diameter 0) (color 0 0 0 0)
@@
     (stroke (width 0) (type default) (color 0 0 0 0))
   )
-  (wire (pts (xy 46.99 115.57) (xy 46.99 120.65))
-    (stroke (width 0) (type default) (color 0 0 0 0))
-  )
   (wire (pts (xy 135.89 115.57) (xy 138.43 115.57))
     (stroke (width 0) (type default) (color 0 0 0 0))
@@
     (stroke (width 0) (type default) (color 0 0 0 0))
   )
-  (polyline (pts (xy 125.73 60.96) (xy 125.73 90.17))
+  (wire (pts (xy 143.51 91.44) (xy 149.86 91.44))
+    (stroke (width 0) (type default) (color 0 0 0 0))
+  )
+  (polyline (pts (xy 125.73 60.96) (xy 125.73 95.25))
     (stroke (width 0) (type default) (color 0 0 0 0))
   )
@@
     (stroke (width 0) (type default) (color 0 0 0 0))
   )
+  (wire (pts (xy 46.99 111.76) (xy 46.99 120.65))
+    (stroke (width 0) (type default) (color 0 0 0 0))
+  )
+  (wire (pts (xy 149.86 83.82) (xy 147.32 83.82))
+    (stroke (width 0) (type default) (color 0 0 0 0))
+  )
   (wire (pts (xy 46.99 115.57) (xy 49.53 115.57))
     (stroke (width 0) (type default) (color 0 0 0 0))
@@
     (stroke (width 0) (type default) (color 0 0 0 0))
   )
-  (polyline (pts (xy 158.75 60.96) (xy 158.75 90.17))
+  (polyline (pts (xy 158.75 60.96) (xy 158.75 95.25))
     (stroke (width 0) (type default) (color 0 0 0 0))
   )
@@
     (stroke (width 0) (type default) (color 0 0 0 0))
   )
-  (polyline (pts (xy 158.75 90.17) (xy 125.73 90.17))
+  (polyline (pts (xy 158.75 95.25) (xy 125.73 95.25))
     (stroke (width 0) (type default) (color 0 0 0 0))
   )
@@
   )
   (wire (pts (xy 121.92 184.15) (xy 121.92 173.99))
+    (stroke (width 0) (type default) (color 0 0 0 0))
+  )
+  (wire (pts (xy 152.4 83.82) (xy 149.86 83.82))
     (stroke (width 0) (type default) (color 0 0 0 0))
   )
@@
     )
   )
-  (global_label "3v3" (shape input) (at 147.32 83.82 0) (fields_autoplaced)
-    (effects (font (size 1.27 1.27)) (justify left))
-    (property "Intersheet References" "${INTERSHEET_REFS}" (id 0) (at 60.96 -40.64 0)
+  (global_label "3v3" (shape input) (at 152.4 83.82 0) (fields_autoplaced)
+    (effects (font (size 1.27 1.27)) (justify left))
+    (property "Intersheet References" "${INTERSHEET_REFS}" (id 0) (at 66.04 -40.64 0)
       (effects (font (size 1.27 1.27)) hide)
     )
@@
     (effects (font (size 1.27 1.27)) (justify right))
     (property "Intersheet References" "${INTERSHEET_REFS}" (id 0) (at 59.69 -62.23 0)
+      (effects (font (size 1.27 1.27)) hide)
+    )
+  )
+  (global_label "GND" (shape input) (at 143.51 91.44 180) (fields_autoplaced)
+    (effects (font (size 1.27 1.27)) (justify right))
+    (property "Intersheet References" "${INTERSHEET_REFS}" (id 0) (at 121.92 8.89 0)
       (effects (font (size 1.27 1.27)) hide)
     )
@@
     (property "Reference" "U7" (id 0) (at 139.7 67.471 0))
     (property "Value" "ATGM336H" (id 1) (at 139.7 70.0079 0))
-    (property "Footprint" "" (id 2) (at 139.7 68.58 0)
+    (property "Footprint" "lora_tracker:ATGM336H" (id 2) (at 139.7 68.58 0)
       (effects (font (size 1.27 1.27)) hide)
     )
@@
     (pin "2")
   )
+  (symbol (lib_id "Device:C") (at 149.86 87.63 0) (unit 1)
+    (in_bom yes) (on_board yes)
+    (property "Reference" "C11" (id 0) (at 153.67 88.9 0)
+      (effects (font (size 1.27 1.27)) (justify left))
+    )
+    (property "Value" "100nF" (id 1) (at 151.13 91.44 0)
+      (effects (font (size 1.27 1.27)) (justify left))
+    )
+    (property "Footprint" "Capacitor_SMD:C_0603_1608Metric_Pad1.08x0.95mm_HandSolder" (id 2) (at 150.8252 91.44 0)
+      (effects (font (size 1.27 1.27)) hide)
+    )
+    (property "Datasheet" "~" (id 3) (at 149.86 87.63 0)
+      (effects (font (size 1.27 1.27)) hide)
+    )
+    (pin "1")
+    (pin "2")
+  )
   (symbol (lib_id "Device:R") (at 118.11 27.94 0) (unit 1)
     (in_bom yes) (on_board yes) (fields_autoplaced)
@@
       (reference "C10") (unit 1) (value "100nF") (footprint "Capacitor_SMD:C_0603_1608Metric_Pad1.08x0.95mm_HandSolder")
     )
+    (path "/cd4ddaf6-f132-4b95-a0be-b45eb04ecd80"
+      (reference "C11") (unit 1) (value "100nF") (footprint "Capacitor_SMD:C_0603_1608Metric_Pad1.08x0.95mm_HandSolder")
+    )
     (path "/c5fb8d0b-52b5-449b-965e-53dc20584b98"
       (reference "J1") (unit 1) (value "ANT") (footprint "Connector_Coaxial:SMA_Samtec_SMA-J-P-X-ST-EM1_EdgeMount")
@@
     )
     (path "/1fde4a5b-e415-4026-82ee-2764bc0d7d81"
-      (reference "U7") (unit 1) (value "ATGM336H") (footprint "")
-    )
-  )
+      (reference "U7") (unit 1) (value "ATGM336H") (footprint "lora_tracker:ATGM336H")
+    )
+  )

Commit message: Update schematics
Parts:
- added J2: Conn_01x02, Connector_PinHeader_2.54mm:PinHeader_2x01_P2.54mm_Vertical_SMD, symbol Connector_Generic:Conn_01x02
Connections:
- new net: J2.1 (Pin_1), U5.9 (SPK-)
- new net: J2.2 (Pin_2), U5.8 (SPK+)
Other:
- moved on the sheet: C11, C7, U6A, U7
