File: extras/schematics/lora_tracker.kicad_sch (KiCad schematic)
At the start: 30 parts, among them J1 ANT, J2 Conn_01x02, J4 Conn_01x03_Female, SW1 SW_Push, SW2 EC11, U1 ESP32, U2 E22-400M30S, U3 RA-01, U4 INP441, U5 MAX98357A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

Commit message: Update schematics
Parts:
- R2: value 1k -> 10k
Changed lines of the file:
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@@
     (in_bom yes) (on_board yes) (fields_autoplaced)
     (property "Reference" "R2" (id 0) (at 106.68 160.3842 90))
-    (property "Value" "1k" (id 1) (at 106.68 162.9211 90))
+    (property "Value" "10k" (id 1) (at 106.68 162.9211 90))
     (property "Footprint" "Resistor_SMD:R_0603_1608Metric_Pad0.98x0.95mm_HandSolder" (id 2) (at 106.68 166.878 90)
       (effects (font (size 1.27 1.27)) hide)
@@
     )
     (path "/ef86053e-dd97-42cd-a0a1-a6dad77f89ec"
-      (reference "R2") (unit 1) (value "1k") (footprint "Resistor_SMD:R_0603_1608Metric_Pad0.98x0.95mm_HandSolder")
+      (reference "R2") (unit 1) (value "10k") (footprint "Resistor_SMD:R_0603_1608Metric_Pad0.98x0.95mm_HandSolder")
     )
     (path "/358feb15-9620-464e-b745-5164d12fcb10"

Commit message: Update schematics
Parts:
- added J3, J5, J6, J7: Conn_01x01, TestPoint:TestPoint_Pad_1.5x1.5mm, symbol Connector_Generic:Conn_01x01
Connections:
- net GND: now also J3.1 (Pin_1), J5.1 (Pin_1), J6.1 (Pin_1), J7.1 (Pin_1)
Other:
- note added: "Screen shield solder pads"
Changed lines of the file:
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@@
   (junction (at 252.73 109.22) (diameter 0) (color 0 0 0 0)
   )
+  (junction (at 146.05 163.83) (diameter 0) (color 0 0 0 0)
+  )
   (junction (at 87.63 115.57) (diameter 0) (color 0 0 0 0)
   )
@@
   )
   (junction (at 193.04 115.57) (diameter 0) (color 0 0 0 0)
+  )
+  (junction (at 146.05 173.99) (diameter 0) (color 0 0 0 0)
+  )
+  (junction (at 146.05 168.91) (diameter 0) (color 0 0 0 0)
   )
   (junction (at 46.99 111.76) (diameter 0) (color 0 0 0 0)
@@
     (stroke (width 0) (type default) (color 0 0 0 0))
   )
+  (wire (pts (xy 146.05 163.83) (xy 149.86 163.83))
+    (stroke (width 0) (type default) (color 0 0 0 0))
+  )
   (wire (pts (xy 36.83 177.8) (xy 49.53 177.8))
     (stroke (width 0) (type default) (color 0 0 0 0))
@@
     (stroke (width 0) (type default) (color 0 0 0 0))
   )
+  (wire (pts (xy 146.05 163.83) (xy 146.05 158.75))
+    (stroke (width 0) (type default) (color 0 0 0 0))
+  )
   (wire (pts (xy 262.89 58.42) (xy 260.35 58.42))
     (stroke (width 0) (type default) (color 0 0 0 0))
@@
     (stroke (width 0) (type default) (color 0 0 0 0))
   )
+  (wire (pts (xy 146.05 168.91) (xy 149.86 168.91))
+    (stroke (width 0) (type default) (color 0 0 0 0))
+  )
   (wire (pts (xy 260.35 88.9) (xy 262.89 88.9))
     (stroke (width 0) (type default) (color 0 0 0 0))
@@
     (stroke (width 0) (type default) (color 0 0 0 0))
   )
+  (polyline (pts (xy 139.7 151.13) (xy 171.45 151.13))
+    (stroke (width 0) (type default) (color 0 0 0 0))
+  )
   (wire (pts (xy 46.99 111.76) (xy 46.99 120.65))
     (stroke (width 0) (type default) (color 0 0 0 0))
@@
     (stroke (width 0) (type default) (color 0 0 0 0))
   )
+  (wire (pts (xy 146.05 173.99) (xy 146.05 168.91))
+    (stroke (width 0) (type default) (color 0 0 0 0))
+  )
   (polyline (pts (xy 175.26 19.05) (xy 175.26 162.56))
     (stroke (width 0) (type default) (color 0 0 0 0))
@@
     (stroke (width 0) (type default) (color 0 0 0 0))
   )
+  (wire (pts (xy 146.05 158.75) (xy 149.86 158.75))
+    (stroke (width 0) (type default) (color 0 0 0 0))
+  )
   (polyline (pts (xy 86.36 146.05) (xy 86.36 193.04))
     (stroke (width 0) (type default) (color 0 0 0 0))
@@
     (stroke (width 0) (type default) (color 0 0 0 0))
   )
+  (polyline (pts (xy 139.7 151.13) (xy 139.7 193.04))
+    (stroke (width 0) (type default) (color 0 0 0 0))
+  )
   (wire (pts (xy 99.06 29.21) (xy 102.87 29.21))
     (stroke (width 0) (type default) (color 0 0 0 0))
@@
     (stroke (width 0) (type default) (color 0 0 0 0))
   )
+  (wire (pts (xy 146.05 180.34) (xy 146.05 173.99))
+    (stroke (width 0) (type default) (color 0 0 0 0))
+  )
   (wire (pts (xy 29.21 72.39) (xy 34.29 72.39))
     (stroke (width 0) (type default) (color 0 0 0 0))
@@
     (stroke (width 0) (type default) (color 0 0 0 0))
   )
+  (polyline (pts (xy 171.45 193.04) (xy 139.7 193.04))
+    (stroke (width 0) (type default) (color 0 0 0 0))
+  )
   (wire (pts (xy 119.38 184.15) (xy 121.92 184.15))
     (stroke (width 0) (type default) (color 0 0 0 0))
@@
     (stroke (width 0) (type default) (color 0 0 0 0))
   )
+  (polyline (pts (xy 171.45 151.13) (xy 171.45 193.04))
+    (stroke (width 0) (type default) (color 0 0 0 0))
+  )
   (wire (pts (xy 49.53 22.86) (xy 49.53 25.4))
     (stroke (width 0) (type default) (color 0 0 0 0))
   )
+  (wire (pts (xy 146.05 173.99) (xy 149.86 173.99))
+    (stroke (width 0) (type default) (color 0 0 0 0))
+  )
   (wire (pts (xy 222.25 120.65) (xy 224.79 120.65))
     (stroke (width 0) (type default) (color 0 0 0 0))
@@
   )
   (wire (pts (xy 58.42 64.77) (xy 63.5 64.77))
+    (stroke (width 0) (type default) (color 0 0 0 0))
+  )
+  (wire (pts (xy 146.05 168.91) (xy 146.05 163.83))
     (stroke (width 0) (type default) (color 0 0 0 0))
   )
@@
   )
   (text "GPS module" (at 135.89 63.5 0)
+    (effects (font (size 1.27 1.27)) (justify left bottom))
+  )
+  (text "Screen shield solder pads" (at 140.97 153.67 0)
     (effects (font (size 1.27 1.27)) (justify left bottom))
   )
@@
     (property "Intersheet References" "${INTERSHEET_REFS}" (id 0) (at 39.4494 30.0223 90)
       (effects (font (size 1.27 1.27)) (justify right) hide)
+    )
+  )
+  (global_label "GND" (shape input) (at 146.05 180.34 270) (fields_autoplaced)
+    (effects (font (size 1.27 1.27)) (justify right))
+    (property "Intersheet References" "${INTERSHEET_REFS}" (id 0) (at 63.5 201.93 0)
+      (effects (font (size 1.27 1.27)) hide)
     )
   )
@@
     )
     (property "Datasheet" "~" (id 3) (at 49.53 22.86 0)
+      (effects (font (size 1.27 1.27)) hide)
+    )
+    (pin "1")
+  )
+  (symbol (lib_id "Connector_Generic:Conn_01x01") (at 154.94 168.91 0) (unit 1)
+    (in_bom yes) (on_board yes) (fields_autoplaced)
+    (property "Reference" "J6" (id 0) (at 156.972 168.0753 0)
+      (effects (font (size 1.27 1.27)) (justify left))
+    )
+    (property "Value" "Conn_01x01" (id 1) (at 156.972 170.6122 0)
+      (effects (font (size 1.27 1.27)) (justify left))
+    )
+    (property "Footprint" "TestPoint:TestPoint_Pad_1.5x1.5mm" (id 2) (at 154.94 168.91 0)
+      (effects (font (size 1.27 1.27)) hide)
+    )
+    (property "Datasheet" "~" (id 3) (at 154.94 168.91 0)
       (effects (font (size 1.27 1.27)) hide)
     )
@@
     (pin "1")
     (pin "2")
+  )
+  (symbol (lib_id "Connector_Generic:Conn_01x01") (at 154.94 173.99 0) (unit 1)
+    (in_bom yes) (on_board yes) (fields_autoplaced)
+    (property "Reference" "J7" (id 0) (at 156.972 173.1553 0)
+      (effects (font (size 1.27 1.27)) (justify left))
+    )
+    (property "Value" "Conn_01x01" (id 1) (at 156.972 175.6922 0)
+      (effects (font (size 1.27 1.27)) (justify left))
+    )
+    (property "Footprint" "TestPoint:TestPoint_Pad_1.5x1.5mm" (id 2) (at 154.94 173.99 0)
+      (effects (font (size 1.27 1.27)) hide)
+    )
+    (property "Datasheet" "~" (id 3) (at 154.94 173.99 0)
+      (effects (font (size 1.27 1.27)) hide)
+    )
+    (pin "1")
+  )
+  (symbol (lib_id "Connector_Generic:Conn_01x01") (at 154.94 158.75 0) (unit 1)
+    (in_bom yes) (on_board yes) (fields_autoplaced)
+    (property "Reference" "J3" (id 0) (at 156.972 157.9153 0)
+      (effects (font (size 1.27 1.27)) (justify left))
+    )
+    (property "Value" "Conn_01x01" (id 1) (at 156.972 160.4522 0)
+      (effects (font (size 1.27 1.27)) (justify left))
+    )
+    (property "Footprint" "TestPoint:TestPoint_Pad_1.5x1.5mm" (id 2) (at 154.94 158.75 0)
+      (effects (font (size 1.27 1.27)) hide)
+    )
+    (property "Datasheet" "~" (id 3) (at 154.94 158.75 0)
+      (effects (font (size 1.27 1.27)) hide)
+    )
+    (pin "1")
   )
   (symbol (lib_id "power:PWR_FLAG") (at 39.37 22.86 0) (unit 1)
@@
     (pin "2")
   )
+  (symbol (lib_id "Connector_Generic:Conn_01x01") (at 154.94 163.83 0) (unit 1)
+    (in_bom yes) (on_board yes) (fields_autoplaced)
+    (property "Reference" "J5" (id 0) (at 156.972 162.9953 0)
+      (effects (font (size 1.27 1.27)) (justify left))
+    )
+    (property "Value" "Conn_01x01" (id 1) (at 156.972 165.5322 0)
+      (effects (font (size 1.27 1.27)) (justify left))
+    )
+    (property "Footprint" "TestPoint:TestPoint_Pad_1.5x1.5mm" (id 2) (at 154.94 163.83 0)
+      (effects (font (size 1.27 1.27)) hide)
+    )
+    (property "Datasheet" "~" (id 3) (at 154.94 163.83 0)
+      (effects (font (size 1.27 1.27)) hide)
+    )
+    (pin "1")
+  )
   (symbol (lib_id "Device:R") (at 106.68 165.1 90) (unit 1)
     (in_bom yes) (on_board yes) (fields_autoplaced)
@@
       (reference "J2") (unit 1) (value "Conn_01x02") (footprint "Connector_PinHeader_2.54mm:PinHeader_2x01_P2.54mm_Vertical_SMD")
     )
+    (path "/88382c4e-7e86-4cdb-96fb-9cd9c2bfd6d8"
+      (reference "J3") (unit 1) (value "Conn_01x01") (footprint "TestPoint:TestPoint_Pad_1.5x1.5mm")
+    )
     (path "/03d94089-9d86-47f6-9c15-68498975a675"
       (reference "J4") (unit 1) (value "Conn_01x03_Female") (footprint "Connector_PinHeader_2.54mm:PinHeader_1x03_P2.54mm_Vertical")
     )
+    (path "/e3d65acf-efc7-4ce6-bf04-e0a44be5be14"
+      (reference "J5") (unit 1) (value "Conn_01x01") (footprint "TestPoint:TestPoint_Pad_1.5x1.5mm")
+    )
+    (path "/59194807-a3e7-42aa-a26f-41b610251c6c"
+      (reference "J6") (unit 1) (value "Conn_01x01") (footprint "TestPoint:TestPoint_Pad_1.5x1.5mm")
+    )
+    (path "/821ab1a8-1423-4faa-be26-25f4b74f7eb3"
+      (reference "J7") (unit 1) (value "Conn_01x01") (footprint "TestPoint:TestPoint_Pad_1.5x1.5mm")
+    )
     (path "/97408edf-4602-44e3-bc11-9f71091e9c9a"
